File: home-mini-v1-drop-in-pcb.kicad_pcb (KiCad board)
At the start: 4 copper layers, 72.4 x 70 mm, 161 parts, among them J1 1775443-2, J2 FH34SRJ-16S-0.5SH_50_, Q1 LBSS138WT1G, Q2 BC847B, Q3 LBSS138WT1G, SW2 BOOT, SW3 SMXS_01K_TP, U1 TPS62130, U10 SN74LVC125APWR, U11 MAX98357AETE_T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

Commit message: error corrections
Parts:
- R46: value 100k -> 68.1k
- renumbered XMOS_DEBUG to XMOS_DEBUG1
Changed lines of the file:
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@@
 			)
 		)
-		(property "Value" "100k"
+		(property "Value" "68.1k"
 			(at 0 1.43 90)
 			(layer "F.Fab")
@@
 			)
 		)
-		(property "LCSC Part #" "C25803"
+		(property "LCSC Part #" "C25976"
 			(at 0 0 270)
 			(unlocked yes)
@@
 			)
 		)
-		(property "Manufacturer Part" "0603WAF1003T5E"
+		(property "Manufacturer Part" "0603WAF6812T5E"
 			(at 0 0 270)
 			(unlocked yes)
@@
 		(descr "surface-mounted straight pin header, 2x10, 1.27mm pitch, double rows")
 		(tags "Surface mounted pin header SMD 2x10 1.27mm double row")
-		(property "Reference" "XMOS_DEBUG"
+		(property "Reference" "XMOS_DEBUG1"
 			(at -3.8 1.1 0)
 			(layer "B.SilkS")
