File: home-mini-v1-drop-in-pcb.kicad_pcb (KiCad board)
At the start: 4 copper layers, 72.4 x 70 mm, 210 parts, among them J1 FH34SRJ-16S-0.5SH_50_, J2 1775443-2, Q1 LBSS138WT1G, Q2 LBSS138WT1G, Q3 BC847B, SW1 SMXS_01K_TP, SW2 BOOT, U1 AP22802AW5-7, U10 SN74LVC125APWR, U11 TLV73333PDBVR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

Commit message: routing
Parts:
- C29, C30, C31, C32, C33: moved to B.Cu
- Y1: footprint Crystal:Crystal_SMD_3225-4Pin_3.2x2.5mm -> Crystal:Crystal_SMD_2016-4Pin_2.0x1.6mm
- moved C4 74.5 mm to (119.6, 111.1)
- moved C5 74.5 mm to (122.0, 108.6)
- moved D1 74.5 mm to (118.6, 111.1)
- moved R2 74.5 mm to (123.5, 113.8)
- moved R3 74.5 mm to (122.5, 113.8)
- moved SW1 74.5 mm to (129.3, 111.8)
- moved U2 74.5 mm to (123.3, 111.1)
- moved R5 74.5 mm to (117.6, 111.1)
- moved C30 40.6 mm to (115.1, 76.4)
- moved C25 40.5 mm to (119.4, 73.4), turned to 90 degrees
- moved C24 40.4 mm to (115.4, 73.9)
- moved Y1 40.4 mm to (117.4, 73.5), turned to 180 degrees
- moved C29 38.7 mm to (114.1, 76.4)
- moved R25 38.2 mm to (107.5, 81.6)
- moved R24 38.2 mm to (107.5, 80.6)
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Routing:
- net ESP_3V3: track 31.5 -> 45.7 mm, vias 5 -> 8
- net Net-(U6-XTAL_N): track 0.00 -> 7.48 mm
- net I2C_SCL: track 0.00 -> 4.46 mm
- net I2C_SDA: track 0.00 -> 4.21 mm
- net Net-(U6-XTAL_P): track 0.00 -> 4.13 mm
- net I2S_MCLK: track 4.36 -> 3.76 mm
- net GND: vias 16 -> 42
