File: home-mini-v1-drop-in-pcb.kicad_pcb (KiCad board)
At the start: 4 copper layers, 72.4 x 70 mm, 210 parts, among them J1 FH34SRJ-16S-0.5SH_50_, J2 1775443-2, Q1 LBSS138WT1G, Q2 LBSS138WT1G, Q3 BC847B, SW1 SMXS_01K_TP, SW2 BOOT, U1 AP22802AW5-7, U10 SN74LVC125APWR, U11 TLV73333PDBVR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

Commit message: routing
Parts:
- removed SW1: SMXS_01K_TP, Onju:SW-SMD_2P-L6.2-W2.5-LS9.4
- added U15: MK-12C02 G1.5, Onju:SW7-SMD-L6.7X2.7X3.2MM, F.Cu at (124.2, 112.8)
