File: power_handling.kicad_sch (KiCad schematic)
At the start: 35 parts, among them J3 Conn_01x08, SW1 SMXS‑01K‑TP, U1 TPS62130, U12 FSUSB42MUX, U2 MIC5365-1.8YC5-TR, U4 MIC5365-0.9YC5-TR

Commit message: routing
Parts:
- removed J3: Conn_01x08, symbol Connector_Generic:Conn_01x08
- added J2: FH34SRJ-16S-0.5SH_50_, Onju:HRS_FH34SRJ-16S-0.5SH_50_, symbol New_Library:FH34SRJ-16S-0.5SH_50_
- U4: value MIC5365-0.9YC5-TR -> TPS7A0309PDBVR; footprint Onju:SOT65P210X110-5N -> Package_TO_SOT_SMD:SOT-23-5; LCSC Part # (none) -> C2977167; MANUFACTURER Micrel -> Texas Instruments; MP MIC5365-0.9YC5-TR -> TPS7A0309PDBVR; Manufacturer (none) -> Texas Instruments; Manufacturer Part (none) -> TPS7A0309PDBVR; Supplier Part (none) -> C2977167
Connections:
- net GND: now also J2.11, J2.2, J2.3, J2.4, J2.5, J2.6, J2.7, J2.8, J2.S1 (SHIELD), J2.S2 (SHIELD)
- net MUTE: now also J2.1
- net USB_D_N: now also D13.2 (A2), J2.10; no longer D14.2 (A2)
- net USB_D_P: now also D14.2 (A2), J2.9; no longer D13.2 (A2)
- net at D15.2 (A2), FB8.1: now also J2.12, J2.13, J2.14, J2.15
- new net RST_BTN: J2.16
Other:
- moved on the sheet: D13, D14, D15, FB8

Commit message: getting ready for production
Connections:
- net GND: now also J2.12, J2.13, J2.14, J2.15; no longer J2.2, J2.3, J2.4, J2.5, J2.6, J2.7
- net MUTE: now also J2.16; no longer J2.1
- net RST_BTN: now also J2.1; no longer J2.16
- net USB_D_N: now also D14.2 (A2), J2.9; no longer D13.2 (A2), J2.10
- net USB_D_P: now also D13.2 (A2), J2.10; no longer D14.2 (A2), J2.9
- new net: D15.2 (A2), FB8.1, J2.2, J2.3, J2.4, J2.5, J2.6, J2.7
Other:
- moved on the sheet: D13, D14, D15, FB8

Commit message: getting ready for production
Parts:
- C10, C7: LCSC Part # (none) -> C913474; Manufacturer (none) -> Murata Electronics; Manufacturer Part (none) -> GRM188Z71A475KE15D
- C12, C8: LCSC Part # (none) -> C49678; Manufacturer (none) -> YAGEO; Manufacturer Part (none) -> CC0805KRX7R9BB104
- C6, C9: LCSC Part # (none) -> C86018; Manufacturer (none) -> Murata Electronics; Manufacturer Part (none) -> GRM188R71A225KE15D
Changed lines of the file:
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@@
+			)
+		)
+		(property "LCSC Part #" "C86018"
+			(at 205.74 97.79 0)
+			(effects
+				(font
+					(size 1.27 1.27)
+				)
+				(hide yes)
+			)
+		)
+		(property "Manufacturer" "Murata Electronics"
+			(at 205.74 97.79 0)
+			(effects
+				(font
+					(size 1.27 1.27)
+				)
+				(hide yes)
+			)
+		)
+		(property "Manufacturer Part" "GRM188R71A225KE15D"
+			(at 205.74 97.79 0)
+			(effects
+				(font
+					(size 1.27 1.27)
+				)
+				(hide yes)
 			)
 		)
@@
 					(size 1.27 1.27)
 				)
+			)
+		)
+		(property "LCSC Part #" "C49678"
+			(at 266.7 140.97 0)
+			(effects
+				(font
+					(size 1.27 1.27)
+				)
+				(hide yes)
+			)
+		)
+		(property "Manufacturer" "YAGEO"
+			(at 266.7 140.97 0)
+			(effects
+				(font
+					(size 1.27 1.27)
+				)
+				(hide yes)
+			)
+		)
+		(property "Manufacturer Part" "CC0805KRX7R9BB104"
+			(at 266.7 140.97 0)
+			(effects
+				(font
+					(size 1.27 1.27)
+				)
+				(hide yes)
 			)
 		)
@@
 			)
 		)
+		(property "LCSC Part #" "C913474"
+			(at 256.54 97.79 0)
+			(effects
+				(font
+					(size 1.27 1.27)
+				)
+				(hide yes)
+			)
+		)
+		(property "Manufacturer" "Murata Electronics"
+			(at 256.54 97.79 0)
+			(effects
+				(font
+					(size 1.27 1.27)
+				)
+				(hide yes)
+			)
+		)
+		(property "Manufacturer Part" "GRM188Z71A475KE15D"
+			(at 256.54 97.79 0)
+			(effects
+				(font
+					(size 1.27 1.27)
+				)
+				(hide yes)
+			)
+		)
 		(pin "1"
 		)
@@
 			)
 		)
+		(property "LCSC Part #" "C49678"
+			(at 266.7 97.79 0)
+			(effects
+				(font
+					(size 1.27 1.27)
+				)
+				(hide yes)
+			)
+		)
+		(property "Manufacturer" "YAGEO"
+			(at 266.7 97.79 0)
+			(effects
+				(font
+					(size 1.27 1.27)
+				)
+				(hide yes)
+			)
+		)
+		(property "Manufacturer Part" "CC0805KRX7R9BB104"
+			(at 266.7 97.79 0)
+			(effects
+				(font
+					(size 1.27 1.27)
+				)
+				(hide yes)
+			)
+		)
 		(pin "1"
 		)
@@
 					(size 1.27 1.27)
 				)
+			)
+		)
+		(property "LCSC Part #" "C86018"
+			(at 205.74 140.97 0)
+			(effects
+				(font
+					(size 1.27 1.27)
+				)
+				(hide yes)
+			)
+		)
+		(property "Manufacturer" "Murata Electronics"
+			(at 205.74 140.97 0)
+			(effects
+				(font
+					(size 1.27 1.27)
+				)
+				(hide yes)
+			)
+		)
+		(property "Manufacturer Part" "GRM188R71A225KE15D"
+			(at 205.74 140.97 0)
+			(effects
+				(font
+					(size 1.27 1.27)
+				)
+				(hide yes)
 			)
 		)
@@
 			)
 		)
+		(property "LCSC Part #" "C913474"
+			(at 256.54 140.97 0)
+			(effects
+				(font
+					(size 1.27 1.27)
+				)
+				(hide yes)
+			)
+		)
+		(property "Manufacturer" "Murata Electronics"
+			(at 256.54 140.97 0)
+			(effects
+				(font
+					(size 1.27 1.27)
+				)
+				(hide yes)
+			)
+		)
+		(property "Manufacturer Part" "GRM188Z71A475KE15D"
+			(at 256.54 140.97 0)
+			(effects
+				(font
+					(size 1.27 1.27)
+				)
+				(hide yes)
+			)
+		)

Commit message: update for production
Parts:
- removed SW1: SMXS‑01K‑TP, Onju:CHS-01TA, symbol New_Library:CHS-01TA
- added SW3: SMXS_01K_TP, Onju:SW-SMD_2P-L6.2-W2.5-LS9.4, symbol Switch:SW_DIP_x01
- C61, C65: LCSC Part # (none) -> C45783; Manufacturer (none) -> Samsung Electro-Mechanics; Manufacturer Part (none) -> CL21A226MAQNNNE
- C62: LCSC Part # (none) -> C15195; Manufacturer (none) -> Samsung Electro-Mechanics; Manufacturer Part (none) -> CL05B103KB5NNNC
- C63: LCSC Part # (none) -> C15850; Manufacturer (none) -> Samsung Electro-Mechanics; Manufacturer Part (none) -> CL21A106KAYNNNE
- C64: LCSC Part # (none) -> C156398; Manufacturer (none) -> FH (Guangdong Fenghua Advanced Tech); Manufacturer Part (none) -> 0603CG221J500NT
- C66: LCSC Part # (none) -> C49678; Manufacturer (none) -> YAGEO; Manufacturer Part (none) -> CC0805KRX7R9BB104
- C75: LCSC Part # (none) -> C1525; Manufacturer (none) -> Samsung Electro-Mechanics; Manufacturer Part (none) -> CL05B104KO5NNNC; Voltage 25V -> 16V
- C76: LCSC Part # (none) -> C14663; Manufacturer (none) -> YAGEO; Manufacturer Part (none) -> CC0603KRX7R9BB104; Voltage 25V -> 50V
- D13, D14, D9: LCSC Part # (none) -> C19626254; Manufacturer (none) -> DOWO; Manufacturer Part (none) -> PESD0402V05
- D15: LCSC Part # (none) -> C48260; Manufacturer (none) -> Texas Instruments; Manufacturer Part (none) -> TPD1E10B06DPYR
- FB8: value 0R -> 30R; LCSC Part # (none) -> C17305; Manufacturer Part (none) -> BLM18PG300SN1D
- L1: LCSC Part # (none) -> C719179; Manufacturer (none) -> BOURNS; Manufacturer Part (none) -> SRP4020TA-2R2M
- R108, R76, R77: LCSC Part # (none) -> C25530; Manufacturer (none) -> UNI-ROYAL(Uniroyal Elec); Manufacturer Part (none) -> 0402WGJ0104TCE
- R14: LCSC Part # (none) -> C25744; Manufacturer (none) -> UNI-ROYAL(Uniroyal Elec); Manufacturer Part (none) -> 0402WGF1002TCE
- R18, R19: LCSC Part # (none) -> C25092; Manufacturer (none) -> UNI-ROYAL(Uniroyal Elec); Manufacturer Part (none) -> 0402WGF220JTCE
- R44: LCSC Part # (none) -> C23185; Manufacturer (none) -> UNI-ROYAL(Uniroyal Elec); Manufacturer Part (none) -> 0603WAF499JT5E
- R46: LCSC Part # (none) -> C25803; Manufacturer (none) -> UNI-ROYAL(Uniroyal Elec); Manufacturer Part (none) -> 0603WAF1003T5E
- R47: LCSC Part # (none) -> C25961; Manufacturer (none) -> UNI-ROYAL(Uniroyal Elec); Manufacturer Part (none) -> 0603WAF2212T5E
- U1: LCSC Part # (none) -> C337502; Manufacturer (none) -> Texas Instruments; Manufacturer Part (none) -> TPS62130ARGTR
- U12: LCSC Part # (none) -> C11355; Manufacturer (none) -> onsemi; Manufacturer Part (none) -> FSUSB42MUX
- U2: LCSC Part # (none) -> C626087; Manufacturer (none) -> Microchip Tech; Manufacturer Part (none) -> MIC5365-1.8YC5-TR
Connections:
- net +3V3: now also SW3.1
- net USB_SEL: now also SW3.2

Commit message: error corrections
Parts:
- R46: value 100k -> 68.1k; LCSC Part # C25803 -> C25976; Manufacturer Part 0603WAF1003T5E -> 0603WAF6812T5E
Changed lines of the file:
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@@
 			)
 		)
-		(property "Value" "100k"
+		(property "Value" "68.1k"
 			(at 243.586 50.546 0)
 			(effects
@@
 			)
 		)
-		(property "LCSC Part #" "C25803"
+		(property "LCSC Part #" "C25976"
 			(at 242.57 50.8 0)
 			(effects
@@
 			)
 		)
-		(property "Manufacturer Part" "0603WAF1003T5E"
+		(property "Manufacturer Part" "0603WAF6812T5E"
 			(at 242.57 50.8 0)
 			(effects

Commit message: prepare for the 1st test batch
Parts:
- removed C10: 4.7uF, Capacitor_SMD:C_0603_1608Metric, symbol Device:C
- removed C12: 100nF, Capacitor_SMD:C_0603_1608Metric, symbol Device:C
- removed C9: 2.2uF, Capacitor_SMD:C_0603_1608Metric, symbol Device:C
- removed U4: TPS7A0309PDBVR, Package_TO_SOT_SMD:SOT-23-5, symbol New_Library:MIC5365-1.8YC5-TR
- added C12, C16, C3, C4: 10uF, Capacitor:C0603, symbol Seeed_libdb:Capacitors/302013252
- added C9: 22pF, Capacitor:C0402, symbol Seeed_libadl:Capacitors/302010018
- added L1: 1uH, Inductor:L2016, symbol Seeed_libdb:Inductor/303011382
- added R11: 51K, Resistor:R0402, symbol Seeed_libadl:Resistors/301010051
- added R12: 100K, Resistor:R0402, symbol Seeed_libadl:Resistors/301010456
- added R5, R6, R7, R8: 0R, Resistor:R0402, symbol Seeed_libadl:Resistors/301010000
- added TP1, TP2: TEST-POINT, Seeed_Misc:TP-D45MIL, symbol 0_Seeed_Misc:TEST-POINT
- added U2: TPS62065DSGR, Ic:DFN8G-0.5-2X2MM, symbol Seeed_libdb:Ic/TPS62065DSGR
- renumbered C75 to C1, C64 to C10, C7 to C11, C65 to C13, C8 to C14, C66 to C15, C76 to C2, C61 to C5, C63 to C6, C62 to C7, C6 to C8, D9 to D1, D13 to D2, D14 to D3, D15 to D4, FB8 to FB1, J2 to J1, L1 to L2, R19 to R1, R77 to R10, R44 to R13, R46 to R14, R47 to R15, R18 to R2, R14 to R3, R76 to R4, R108 to R9, SW3 to SW1, U12 to U1, U1 to U3, U2 to U4
Connections:
- net +5V: now also C3.1, C4.1, R5.1, R7.1, U2.7 (AVIN), U2.8 (PVIN)
- net GND: now also C12.2, C16.2, C3.2, C4.2, R12.1, R8.1, TP2.1 (T), U2.1 (PGND), U2.3 (AGND), U2.9 (PAD)
- new net: C9.2, R11.1, R12.2, U2.4 (FB)
- new net: R7.2, R8.2, U2.6 (MODE)
- new net: L1.1, U2.2 (SW)
- new net: R5.2, R6.2, U2.5 (EN)
- new net 0.9V: C12.1, C16.1, C9.1, L1.2, R11.2, TP1.1 (T)
- new net 3V3_PG: R6.1
Other:
- moved on the sheet: C11, C14, C8, U4
