File: power_handling.kicad_sch (KiCad schematic)
At the start: 60 parts, among them J1 FH34SRJ-16S-0.5SH_50_, SW1 SMXS_01K_TP, U1 AP22802AW5-7, U2 FSUSB42MUX, U3 TPS62827DMQR, U4 TPS62065DSGR, U5 ME6211C18M5G-N

Commit message: prepare for the 1st test batch
Connections:
- net 0.9V renamed +0V9
Changed lines of the file:
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@@
 			)
 		)
-		(property "Value" "0.9V"
+		(property "Value" "+0V9"
 			(at 270.51 122.428 0)
 			(effects

Commit message: routing
Parts:
- removed SW1: SMXS_01K_TP, Onju:SW-SMD_2P-L6.2-W2.5-LS9.4, symbol Switch:SW_DIP_x01
- added U15: MK-12C02 G1.5, Onju:SW7-SMD-L6.7X2.7X3.2MM, symbol New_Library:MK-12C02_G1.5
Connections:
- net +3V3: now also U15.3 (B)
- net GND: now also U15.P1 (SS2), U15.P2 (SS2), U15.P3 (SS2), U15.P4 (SS2)
- net USB_SEL: now also U15.2 (COM)
- no-connect marks 1 -> 2
Changed lines of the file:
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@@
 	)
 	(no_connect
+		(at 20.32 173.99)
+	)
+	(no_connect
 		(at 240.03 90.17)
 	)
@@
 	(wire
 		(pts
-			(xy 252.73 26.67) (xy 252.73 30.48)
+			(xy 25.4 180.34) (xy 25.4 184.15)
 		)
 		(stroke
@@
 	(wire
 		(pts
-			(xy 50.8 48.26) (xy 53.34 48.26)
+			(xy 252.73 26.67) (xy 252.73 30.48)
 		)
 		(stroke
@@
 	(wire
 		(pts
-			(xy 45.72 168.91) (xy 60.96 168.91)
+			(xy 50.8 48.26) (xy 53.34 48.26)
 		)
 		(stroke
@@
 	(wire
 		(pts
-			(xy 148.59 30.48) (xy 167.64 30.48)
+			(xy 45.72 168.91) (xy 60.96 168.91)
 		)
 		(stroke
@@
 	(wire
 		(pts
-			(xy 57.15 176.53) (xy 60.96 176.53)
+			(xy 148.59 30.48) (xy 167.64 30.48)
 		)
 		(stroke
@@
 	(wire
 		(pts
-			(xy 71.12 149.86) (xy 58.42 149.86)
+			(xy 57.15 176.53) (xy 60.96 176.53)
 		)
 		(stroke
@@
 	(wire
 		(pts
-			(xy 251.46 85.09) (xy 251.46 88.9)
+			(xy 71.12 149.86) (xy 58.42 149.86)
 		)
 		(stroke
@@
 	(wire
 		(pts
-			(xy 50.8 45.72) (xy 53.34 45.72)
+			(xy 251.46 85.09) (xy 251.46 88.9)
 		)
 		(stroke
@@
 	(wire
 		(pts
-			(xy 33.02 176.53) (xy 39.37 176.53)
+			(xy 50.8 45.72) (xy 53.34 45.72)
 		)
 		(stroke
@@
 	(wire
 		(pts
-			(xy 16.51 175.26) (xy 16.51 176.53)
+			(xy 16.51 177.8) (xy 16.51 179.07)
 		)
 		(stroke
@@
 	(wire
 		(pts
+			(xy 27.94 176.53) (xy 39.37 176.53)
+		)
+		(stroke
+			(width 0)
+			(type default)
+		)
+	)
+	(wire
+		(pts
 			(xy 53.34 30.48) (xy 53.34 33.02)
 		)
@@
 	(wire
 		(pts
-			(xy 16.51 176.53) (xy 17.78 176.53)
+			(xy 16.51 179.07) (xy 20.32 179.07)
 		)
 		(stroke
@@
 	)
 	(symbol
+		(lib_id "power:GND")
+		(at 25.4 184.15 0)
+		(unit 1)
+		(exclude_from_sim no)
+		(in_bom yes)
+		(on_board yes)
+		(dnp no)
+		(fields_autoplaced yes)
+		(property "Reference" "#PWR0195"
+			(at 25.4 190.5 0)
+			(effects
+				(font
+					(size 1.27 1.27)
+				)
+				(hide yes)
+			)
+		)
+		(property "Value" "GND"
+			(at 25.4 189.23 0)
+			(effects
+				(font
+					(size 1.27 1.27)
+				)
+			)
+		)
+		(property "Footprint" ""
+			(at 25.4 184.15 0)
+			(effects
+				(font
+					(size 1.27 1.27)
+				)
+				(hide yes)
+			)
+		)
+		(property "Datasheet" ""
+			(at 25.4 184.15 0)
+			(effects
+				(font
+					(size 1.27 1.27)
+				)
+				(hide yes)
+			)
+		)
+		(property "Description" "Power symbol creates a global label with name \"GND\" , ground"
+			(at 25.4 184.15 0)
+			(effects
+				(font
+					(size 1.27 1.27)
+				)
+				(hide yes)
+			)
+		)
+		(pin "1"
+		)
+		(instances
+			(project ""
+				(path "/204e071a-14ed-47a0-be54-332ac2b951cf/1e1926d7-db4f-450f-be85-739e9691d6cf"
+					(reference "#PWR0195")
+					(unit 1)
+				)
+			)
+		)
+	)
+	(symbol
 		(lib_id "0_Seeed_Misc:TEST-POINT")
 		(at 251.46 80.01 90)
@@
 	)
 	(symbol
+		(lib_id "New_Library:MK-12C02_G1.5")
+		(at 25.4 186.69 0)
+		(mirror y)
+		(unit 1)
+		(exclude_from_sim no)
+		(in_bom yes)
+		(on_board yes)
+		(dnp no)
+		(property "Reference" "U15"
+			(at 24.4348 170.18 0)
+			(effects
+				(font
+					(size 1.27 1.27)
+				)
+			)
+		)
+		(property "Value" "MK-12C02 G1.5"
+			(at 27.686 172.466 0)
+			(effects
+				(font
+					(size 1.27 1.27)
+				)
+			)
+		)
+		(property "Footprint" "Onju:SW7-SMD-L6.7X2.7X3.2MM"
+			(at 25.4 186.69 0)
+			(effects
+				(font
+					(size 1.27 1.27)
+				)
+				(hide yes)
+			)
+		)
+		(property "Datasheet" ""
+			(at 25.4 186.69 0)
+			(effects
+				(font
+					(size 1.27 1.27)
+				)
+				(hide yes)
+			)
+		)
+		(property "Description" ""
+			(at 25.4 186.69 0)
+			(effects
+				(font
+					(size 1.27 1.27)
+				)
+				(hide yes)
+			)
+		)
+		(property "Manufacturer" "G-Switch"
+			(at 25.4 186.69 0)
+			(effects
+				(font
+					(size 1.27 1.27)
+				)
+				(hide yes)
+			)
+		)
+		(property "Manufacturer part #" "MK-12C02-G015"
+			(at 25.4 186.69 0)
+			(effects
+				(font
+					(size 1.27 1.27)
+				)
+				(hide yes)
+			)
+		)
+		(property "LCSC part #" "C2911519"
+			(at 25.4 186.69 0)
+			(effects
+				(font
+					(size 1.27 1.27)
+				)
+				(hide yes)
+			)
+		)
+		(pin "P1"
+		)
+		(pin "2"
+		)
+		(pin "1"
+		)
+		(pin "P2"
+		)
+		(pin "P4"
+		)
+		(pin "3"
+		)
+		(pin "P3"
+		)
+		(instances
+			(project ""
+				(path "/204e071a-14ed-47a0-be54-332ac2b951cf/1e1926d7-db4f-450f-be85-739e9691d6cf"
+					(reference "U15")
+					(unit 1)
+				)
+			)
+		)
+	)
+	(symbol
 		(lib_id "Seeed_libadl:Capacitors/302010024")
 		(at 167.64 52.07 0)
@@
 	(symbol
 		(lib_id "power:+3V3")
-		(at 16.51 175.26 0)
+		(at 16.51 177.8 0)
 		(unit 1)
 		(exclude_from_sim no)
@@
 		(fields_autoplaced yes)
 		(property "Reference" "#PWR02"
-			(at 16.51 179.07 0)
+			(at 16.51 181.61 0)
 			(effects
 				(font
@@
 		)
 		(property "Value" "+3V3"
-			(at 16.51 170.18 0)
+			(at 16.51 172.72 0)
 			(effects
 				(font
@@
 		)
 		(property "Footprint" ""
-			(at 16.51 175.26 0)
+			(at 16.51 177.8 0)
 			(effects
 				(font
@@
 		)
 		(property "Datasheet" ""
-			(at 16.51 175.26 0)
+			(at 16.51 177.8 0)
 			(effects
 				(font
@@
 		)
 		(property "Description" "Power symbol creates a global label with name \"+3V3\""
-			(at 16.51 175.26 0)
+			(at 16.51 177.8 0)
 			(effects
 				(font
@@
 					(unit 1)
 				)
-			)
-		)
-	)
-	(symbol
-		(lib_id "Switch:SW_DIP_x01")
-		(at 25.4 176.53 0)
-		(unit 1)
-		(exclude_from_sim no)
-		(in_bom yes)
-		(on_board yes)
-		(dnp no)
-		(property "Reference" "SW1"
-			(at 25.4 170.942 0)
-			(effects
-				(font
-					(size 1.27 1.27)
-				)
-			)
-		)
-		(property "Value" "SMXS_01K_TP"
-			(at 25.4 172.72 0)
-			(effects
-				(font
-					(size 1.27 1.27)
-				)
-			)
-		)
-		(property "Footprint" "Onju:SW-SMD_2P-L6.2-W2.5-LS9.4"
-			(at 25.4 176.53 0)
-			(effects
-				(font
-					(size 1.27 1.27)
-				)
-				(hide yes)
-			)
-		)
-		(property "Datasheet" "~"
-			(at 25.4 176.53 0)
-			(effects
-				(font
-					(size 1.27 1.27)
-				)
-				(hide yes)
-			)
-		)
-		(property "Description" "1x DIP Switch, Single Pole Single Throw (SPST) switch, small symbol"
-			(at 25.4 176.53 0)
-			(effects
-				(font
-					(size 1.27 1.27)
-				)
-				(hide yes)
-			)
-		)
-		(property "MANUFACTURER" "SM Switch"
-			(at 25.4 176.53 0)
-			(effects
-				(font
-					(size 1.27 1.27)
-				)
-				(hide yes)
-			)
-		)
-		(property "MP" "SMXS-01K-TP"
-			(at 25.4 176.53 0)
-			(effects
-				(font
-					(size 1.27 1.27)
-				)
-				(hide yes)
-			)
-		)
-		(property "Manufacturer" "SM Switch"
-			(at 25.4 176.53 0)
-			(effects
-				(font
-					(size 1.27 1.27)
-				)
-				(hide yes)
-			)
-		)
-		(property "Manufacturer Part" "SMXS-01K-TP"
-			(at 25.4 176.53 0)
-			(effects
-				(font
-					(size 1.27 1.27)
-				)
-				(hide yes)
-			)
-		)
-		(property "Supplier Part" "C5439760"
-			(at 25.4 176.53 0)
-			(effects
-				(font
-					(size 1.27 1.27)
-				)
-				(hide yes)
-			)
-		)
-		(property "LCSC Part #" "C5439760"
-			(at 25.4 176.53 0)
-			(effects
-				(font
-					(size 1.27 1.27)
-				)
-				(hide yes)
-			)
-		)
-		(pin "1"
-		)
-		(pin "2"
-		)
-		(instances
-			(project "home-mini-v1-drop-in-pcb"
-				(path "/204e071a-14ed-47a0-be54-332ac2b951cf/1e1926d7-db4f-450f-be85-739e9691d6cf"
-					(reference "SW1")
-					(unit 1)
-				)

Commit message: routing
Parts:
- TP1: footprint Seeed_Misc:TP-D45MIL -> TestPoint:TestPoint_Pad_D1.0mm
Changed lines of the file:
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@@
 			)
 		)
-		(property "Footprint" "Seeed_Misc:TP-D45MIL"
+		(property "Footprint" "TestPoint:TestPoint_Pad_D1.0mm"
 			(at 86.36 95.25 0)
 			(effects

Commit message: routing done
Parts:
- R8: footprint Capacitor_SMD:C_0402_1005Metric -> Resistor_SMD:R_0402_1005Metric
- renumbered U15 to SW1

Commit message: ready for the 1st test batch
Parts:
- C1: LCSC Part # (none) -> C9196; Manufacturer YAGEO -> FH (Guangdong Fenghua Advanced Tech); Manufacturer Part (none) -> 1206B102K202NT; Voltage (none) -> 2kV
- C10, C18, C21, C9: LCSC Part # (none) -> C19702; Manufacturer Samsung -> Samsung Electro-Mechanics; Manufacturer Part (none) -> CL10A106KP8NNNC; Voltage (none) -> 10V
- C12, C16: LCSC Part # (none) -> C43922; Manufacturer YAGEO -> FH (Guangdong Fenghua Advanced Tech); Manufacturer Part (none) -> 0603B225K160NT; Voltage (none) -> 16V
- C14: LCSC Part # (none) -> C40059; Manufacturer YAGEO -> FH (Guangdong Fenghua Advanced Tech); Manufacturer Part (none) -> 0402CG121J500NT; Voltage (none) -> 50V
- C15: Dielectric C0G -> NP0; LCSC Part # (none) -> C1555; Manufacturer YAGEO -> FH (Guangdong Fenghua Advanced Tech); Manufacturer Part (none) -> 0402CG220J500NT; Voltage (none) -> 50V
- C17: LCSC Part # (none) -> C45783; Manufacturer Samsung -> Samsung Electro-Mechanics; Manufacturer Part (none) -> CL21A226MAQNNNE; Voltage (none) -> 25V
- C19: LCSC Part # (none) -> C1525; Manufacturer YAGEO -> Samsung Electro-Mechanics; Manufacturer Part (none) -> CL05B104KO5NNNC; Voltage (none) -> 16V
- C20: LCSC Part # (none) -> C14663; Manufacturer Part (none) -> CC0603KRX7R9BB104; Voltage (none) -> 50V
- J1: LCSC Part # (none) -> C324725; Manufacturer (none) -> HRS(Hirose); Manufacturer Part (none) -> FH34SRJ-16S-0.5SH(50)
- L1: value 0.47uH -> 470nH; footprint OPL_Inductor:L0805 -> OPL_Inductor:L0806; LCSC Part # (none) -> C97014; Manufacturer Part (none) -> WPN201610MR47MT
- L2: LCSC Part # (none) -> C395545; Manufacturer Part (none) -> WPN201610U1R0MTY01
- R1: LCSC Part # (none) -> C107699; Manufacturer Part (none) -> RC0805JR-071ML
- R10, R12, R14, R6: LCSC Part # (none) -> C17168; Manufacturer YAGEO -> UNI-ROYAL(Uniroyal Elec); Manufacturer Part (none) -> 0402WGF0000TCE
- R16: LCSC Part # (none) -> C25092; Manufacturer YAGEO -> UNI-ROYAL(Uniroyal Elec); Manufacturer Part (none) -> 0402WGF220JTCE
- R17, R20, R8, R9: LCSC Part # (none) -> C25530; Manufacturer YAGEO -> UNI-ROYAL(Uniroyal Elec); Manufacturer Part (none) -> 0402WGJ0104TCE
- R18: LCSC Part # (none) -> C43473; Manufacturer YAGEO -> UNI-ROYAL(Uniroyal Elec); Manufacturer Part (none) -> 0402WGF2212TCE
- R19: LCSC Part # (none) -> C25794; Manufacturer YAGEO -> UNI-ROYAL(Uniroyal Elec); Manufacturer Part (none) -> 0402WGF5102TCE
- SW1: LCSC Part # (none) -> C20611677; Manufacturer G-Switch -> HOOYA; Manufacturer Part (none) -> MK-12C02G1.5-W
- U3: LCSC Part # (none) -> C2071448; Manufacturer TI -> Texas Instruments; Manufacturer Part (none) -> TPS62827DMQR
- U4: LCSC Part # (none) -> C398352; Manufacturer TI -> Texas Instruments; Manufacturer Part (none) -> TPS62065DSGR
- U5: LCSC Part # (none) -> C236671; Manufacturer (none) -> MICRONE(Nanjing Micro One Elec); Manufacturer Part (none) -> ME6211C18M5G-N

Commit message: mods after 1st batch testing
Connections:
- net GND: now also J1.2, J1.3, J1.4, J1.5, J1.6, J1.9; no longer J1.11, J1.12, J1.13, J1.14, J1.15, J1.8
- net MUTE: now also J1.1; no longer J1.16
- net RST_BTN: now also J1.16; no longer J1.1
- net USB_D_N: now also D2.2 (A2), J1.8; no longer D3.2 (A2), J1.9
- net USB_D_P: now also D3.2 (A2), J1.7; no longer D2.2 (A2), J1.10
- new net: D4.2 (A2), FB1.1, J1.10, J1.11, J1.12, J1.13, J1.14, J1.15
Other:
- moved on the sheet: D2, D3, D4, FB1

Commit message: final mods before production
Parts:
- FB1: footprint Onju:TPD1E05U06DPYR -> Onju:BLM18PG300SN1D
Changed lines of the file:
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@@
 			)
 		)
-		(property "Footprint" "Onju:TPD1E05U06DPYR"
+		(property "Footprint" "Onju:BLM18PG300SN1D"
 			(at 92.71 27.178 90)
 			(effects
@@
 		)
 		(property "Current" "6A"
-			(at 92.71 33.782 90)
+			(at 92.71 29.464 90)
 			(effects
 				(font
