File: power_handling.kicad_sch (KiCad schematic)
At the start: 52 parts, among them J1 FH34SRJ-16S-0.5SH_50_, U1 AP22802AW5-7, U3 TPS62827DMQR, U4 TPS62065DSGR, U5 ME6211C18M5G-N

Commit message: pcb antenna finetuning
Parts:
- added TP18: MUTE, TestPoint:TestPoint_Pad_D1.0mm, symbol Connector:TestPoint
Connections:
- net MUTE: now also TP18.1
Changed lines of the file:
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@@
 	)
 	(junction
+		(at 52.07 60.96)
+		(diameter 0)
+		(color 0 0 0 0)
+	)
+	(junction
 		(at 48.26 106.68)
 		(diameter 0)
@@
 	(wire
 		(pts
+			(xy 52.07 60.96) (xy 53.34 60.96)
+		)
+		(stroke
+			(width 0)
+			(type default)
+		)
+	)
+	(wire
+		(pts
 			(xy 220.98 142.24) (xy 220.98 149.86)
 		)
@@
 	(wire
 		(pts
-			(xy 50.8 60.96) (xy 53.34 60.96)
+			(xy 50.8 60.96) (xy 52.07 60.96)
 		)
 		(stroke
@@
 					(unit 1)
 				)
+			)
+		)
+	)
+	(symbol
+		(lib_id "Connector:TestPoint")
+		(at 52.07 60.96 180)
+		(unit 1)
+		(exclude_from_sim no)
+		(in_bom no)
+		(on_board yes)
+		(dnp yes)
+		(property "Reference" "TP18"
+			(at 50.038 66.548 0)
+			(effects
+				(font
+					(size 1.27 1.27)
+				)
+				(justify right)
+			)
+		)
+		(property "Value" "MUTE"
+			(at 54.61 65.5319 0)
+			(effects
+				(font
+					(size 1.27 1.27)
+				)
+				(justify right)
+				(hide yes)
+			)
+		)
+		(property "Footprint" "TestPoint:TestPoint_Pad_D1.0mm"
+			(at 46.99 60.96 0)
+			(effects
+				(font
+					(size 1.27 1.27)
+				)
+				(hide yes)
+			)
+		)
+		(property "Datasheet" "~"
+			(at 46.99 60.96 0)
+			(effects
+				(font
+					(size 1.27 1.27)
+				)
+				(hide yes)
+			)
+		)
+		(property "Description" "test point"
+			(at 52.07 60.96 0)
+			(effects
+				(font
+					(size 1.27 1.27)
+				)
+				(hide yes)
+			)
+		)
+		(pin "1"
+		)
+		(instances
+			(project ""
+				(path "/204e071a-14ed-47a0-be54-332ac2b951cf/1e1926d7-db4f-450f-be85-739e9691d6cf"
+					(reference "TP18")
+					(unit 1)
+				)

Commit message: v2 hardware revision
MPR121 touch controller added to replace esp32-s3 integrated touch pins
Parts:
- removed C11, C13: 100nF, Capacitor_SMD:C_0402_1005Metric, symbol Seeed_libadl:Capacitors/302010024
- removed C7, C8: 10uF, Capacitor_SMD:C_0603_1608Metric, symbol Seeed_libdb:Capacitors/302013252
- removed R11, R13, R15, R7: 0R, Resistor_SMD:R_0402_1005Metric, symbol Seeed_libadl:Resistors/301010000
- added TP10: TEST-POINT, TestPoint:TestPoint_Pad_D3.0mm, symbol 0_Seeed_Misc:TEST-POINT
- C1: Function (none) -> POWER; SKU 302010189 -> (none); Status BeagleBone Carrier Board -> (none)
- C10, C18, C21, C9: Function (none) -> POWER; SKU 302013252 -> (none)
- C12, C16: Function (none) -> POWER; SKU 302010054 -> (none)
- C14: Function (none) -> POWER; SKU 302013487 -> (none); Status Frame 2 EVT -> (none)
- C15: Function (none) -> POWER; SKU 302010018 -> (none)
- C17: Function (none) -> POWER; SKU 302013260 -> (none)
- C19: Function (none) -> POWER; SKU 302010024 -> (none)
- C2: Supplier Part C913474 -> (none)
- C20: Function (none) -> POWER; SKU 302010138 -> (none)
- C3, C6: Supplier Part C14663 -> (none)
- FB1: Part number BLM18PG300SN1D -> (none)
- J1: Availability In Stock -> (none); Check_prices https://www.snapeda.com/parts/FH34SRJ-16S-0.5SH(50)/Hirose/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 -> (none); Function (none) -> POWER
- L1: Function (none) -> POWER; SKU 303010172 -> (none); Status BeagleBone Carrier Board -> (none)
- L2: Function (none) -> POWER; SKU 303011382 -> (none)
- R1: Function (none) -> POWER; SKU 301010321 -> (none); Status Combox Pro -> (none)
- R10, R12, R14, R6: Function (none) -> POWER; SKU 301010000 -> (none)
- R16: SKU 301010002 -> (none); Status BeagleBone Carrier Board -> (none)
- R17, R8, R9: Function (none) -> POWER; SKU 301010456 -> (none); Status BeagleBone Carrier Board -> (none)
- R18: Function (none) -> POWER; SKU 301011331 -> (none); Status Zola Gateway -> (none)
- R19: Function (none) -> POWER; SKU 301013788 -> (none)
- R20: Function (none) -> POWER; SKU 301010456 -> (none)
- R4: Supplier Part C25530 -> (none)
- TP5: footprint TestPoint:TestPoint_Pad_D1.0mm -> TestPoint:TestPoint_Pad_D3.0mm
- U1: Function (none) -> POWER; Supplier LCSC -> (none); Supplier Part C211404 -> (none)
- U3: Function (none) -> POWER; SKU 310033232 -> (none)
- U4: Function (none) -> POWER; SKU 310033233 -> (none); Status Voice Kit -> (none)
- U5: Function (none) -> POWER
Connections:
- net +5V: now also TP10.1 (T)
Other:
- moved on the sheet: R10, R6
