File: xmos.kicad_sch (KiCad schematic)
At the start: 69 parts, among them Q1 LBSS138WT1G, Q2 BC847B, Q3 LBSS138WT1G, U10 SN74LVC125APWR, U7 XU316-1024-QF60B-C24, U8 W25Q128JVSIQ, U9 TLV73333PDBVR, Y2 24MHz

Commit message: routing
Parts:
- added C142, C143: 100nF, Capacitor_SMD:C_0402_1005Metric, symbol Seeed_libadl:Capacitors/302010024
- added J5: ~, Connector_PinHeader_1.27mm:PinHeader_2x10_P1.27mm_Vertical_SMD, symbol Seeed_libdb:Connector/1.27Header
- added R1, R2: 22R, Resistor_SMD:R_0402_1005Metric, symbol Seeed_libdb:Resistors/301010002
- U8: value W25Q128JVSIQ -> W25Q32JVSSIQ
Connections:
- net +1V8: now also C142.1, J5.1
- net GND: now also C142.2, C143.2, J5.13, J5.15, J5.17, J5.19, J5.3, J5.5, J5.7, J5.9
- net RST_N: now also J5.10
- net TCK: now also J5.4
- net TDI: now also J5.8
- net TDO: now also J5.6
- net TMS: now also J5.2
- net VDDIO: now also C143.1, J5.11
- net XL_DN1: now reaches U7.33 (X1D16)
- net XL_DN1: now also J5.12
- net XL_DN0: now reaches U7.35 (X1D17)
- net XL_DN0: now also J5.14
- net at U7.36 (X1D18): now also R1.1
- net at U7.37 (X1D19): now also R2.1
- net ESP_IO40: no longer names the net of U7.51 (X0D43)
- net ESP_IO41: no longer names the net of U7.58 (X0D33)
- net I2C2_SCL: no longer names the net of U7.40 (X0D29)
- net I2C2_SDA: no longer names the net of U7.54 (X0D30)
- net I2S_BCLK: no longer names the net of U7.13 (X1D10)
- net I2S_DIN_ESP: no longer names the net of U7.53 (X1D34)
- net I2S_DIN_SEC: no longer names the net of U7.9 (X1D00)
- net I2S_LRCK: no longer names the net of U7.10 (X1D01)
- net I2S_MCLK: no longer names the net of U7.14 (X1D11)
- net RST_DAC: no longer names the net of U7.56 (X0D32)
- net XMOS_MUTE_DET: no longer names the net of U7.46 (X0D40)
- net XOD31: no longer names the net of U7.55 (X0D31)
- new net XL_UP0: J5.16, R1.2
- new net XL_UP1: J5.18, R2.2
- no-connect marks 8 -> 17

Commit message: getting ready for production
Parts:
- C59: LCSC Part # (none) -> C86018; Manufacturer (none) -> Murata Electronics; Manufacturer Part (none) -> GRM188R71A225KE15D
- Q1: footprint Onju:SC-70-3_L2.1-W1.3-P0.65-LS2.1-BR -> Package_TO_SOT_SMD:SOT-323_SC-70
Changed lines of the file:
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@@
 			)
 		)
+		(property "LCSC Part #" "C86018"
+			(at 175.26 130.81 0)
+			(effects
+				(font
+					(size 1.27 1.27)
+				)
+				(hide yes)
+			)
+		)
+		(property "Manufacturer" "Murata Electronics"
+			(at 175.26 130.81 0)
+			(effects
+				(font
+					(size 1.27 1.27)
+				)
+				(hide yes)
+			)
+		)
+		(property "Manufacturer Part" "GRM188R71A225KE15D"
+			(at 175.26 130.81 0)
+			(effects
+				(font
+					(size 1.27 1.27)
+				)
+				(hide yes)
+			)
+		)
 		(pin "1"
 		)
@@
 			)
 		)
-		(property "Footprint" "Onju:SC-70-3_L2.1-W1.3-P0.65-LS2.1-BR"
+		(property "Footprint" "Package_TO_SOT_SMD:SOT-323_SC-70"
 			(at 152.4 196.85 0)
 			(effects

Commit message: update for production
Parts:
- C142, C143: Dielectric (none) -> X5R; LCSC Part # (none) -> C1525
- C37, C38, C39, C40, C41, C42, C43, C45, C46, C47, C48, C49, C50, C51, C52, C56, C57, C58, C67, C68, C69, C70: LCSC Part # (none) -> C1525; Manufacturer (none) -> Samsung Electro-Mechanics; Manufacturer Part (none) -> CL05B104KO5NNNC; Voltage 25V -> 16V
- C44, C53, C60: LCSC Part # (none) -> C52923; Manufacturer (none) -> Samsung Electro-Mechanics; Manufacturer Part (none) -> CL05A105KA5NQNC; Voltage 10V -> 25V
- C54, C55: LCSC Part # (none) -> C1548; Manufacturer (none) -> FH (Guangdong Fenghua Advanced Tech); Manufacturer Part (none) -> 0402CG150J500NT
- D2: LCSC Part # (none) -> C27636108; Manufacturer (none) -> ON SEMICONDUCTOR; Manufacturer Part (none) -> RB521S30T1G
- D3, D4, D5, D6, D7, D8: LCSC Part # (none) -> C19626254; Manufacturer (none) -> DOWO; Manufacturer Part (none) -> PESD0402V05
- FB2: LCSC Part # (none) -> C14709; Manufacturer Part (none) -> BLM18PG121SN1D
- FB3, FB4: LCSC Part # (none) -> C85833; Manufacturer Part (none) -> BLM18KG601SN1D
- MK1, MK2: LCSC Part # (none) -> C3171752; Manufacturer (none) -> TDK InvenSense; Manufacturer Part (none) -> MMICT390200012
- Q1: LCSC Part # (none) -> C383201; Manufacturer LRC(乐山无线电) -> LRC
- Q2: LCSC Part # (none) -> C20069135; Manufacturer (none) -> hongjiacheng; Manufacturer Part (none) -> BC847B
- R1, R2: LCSC Part # (none) -> C25092; Manufacturer YAGEO -> UNI-ROYAL(Uniroyal Elec); Manufacturer Part (none) -> 0402WGF220JTCE
- R10, R11, R12, R13, R51, R6: LCSC Part # (none) -> C25076; Manufacturer (none) -> UNI-ROYAL(Uniroyal Elec); Manufacturer Part (none) -> 0402WGF1000TCE
- R29, R4, R55: LCSC Part # (none) -> C25792; Manufacturer (none) -> UNI-ROYAL(Uniroyal Elec); Manufacturer Part (none) -> 0402WGF4702TCE
- R30: LCSC Part # (none) -> C25530; Manufacturer (none) -> UNI-ROYAL(Uniroyal Elec); Manufacturer Part (none) -> 0402WGJ0104TCE
- R31: LCSC Part # (none) -> C25130; Manufacturer (none) -> UNI-ROYAL(Uniroyal Elec); Manufacturer Part (none) -> 0402WGF6800TCE
- R32: LCSC Part # (none) -> C26083; Manufacturer (none) -> UNI-ROYAL(Uniroyal Elec); Manufacturer Part (none) -> 0402WGF1004TCE
- R5: LCSC Part # (none) -> C25744; Manufacturer (none) -> UNI-ROYAL(Uniroyal Elec); Manufacturer Part (none) -> 0402WGF1002TCE
- R50: LCSC Part # (none) -> C25900; Manufacturer (none) -> UNI-ROYAL(Uniroyal Elec); Manufacturer Part (none) -> 0402WGF4701TCE
- R52: LCSC Part # (none) -> C11702; Manufacturer (none) -> UNI-ROYAL(Uniroyal Elec); Manufacturer Part (none) -> 0402WGF1001TCE
- R53: LCSC Part # (none) -> C25790; Manufacturer (none) -> UNI-ROYAL(Uniroyal Elec); Manufacturer Part (none) -> 0402WGF4703TCE
- R54: LCSC Part # (none) -> C25890; Manufacturer (none) -> UNI-ROYAL(Uniroyal Elec); Manufacturer Part (none) -> 0402WGF3301TCE
- U10: LCSC Part # (none) -> C7813; Manufacturer (none) -> Texas Instruments; Manufacturer Part (none) -> SN74LVC125APWR
- U7: LCSC Part # (none) -> C6617472; Manufacturer (none) -> XMOS; Manufacturer Part (none) -> XU316-1024-QF60B-C24
- U8: Manufacturer (none) -> Winbond Elec
- U9: LCSC Part # (none) -> C134139; Manufacturer (none) -> Texas Instruments; Manufacturer Part (none) -> TLV73333PDBVR
- Y2: LCSC Part # (none) -> C70590; Manufacturer (none) -> YXC Crystal Oscillators; Manufacturer Part (none) -> X322524MOB4SI

Commit message: update for production
Parts:
- renumbered J5 to XMOS_DEBUG1
Changed lines of the file:
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@@
 		(on_board yes)
 		(dnp no)
-		(property "Reference" "J5"
+		(property "Reference" "XMOS_DEBUG1"
 			(at 68.58 135.89 0)
 			(effects
@@
 			(project "home-mini-v1-drop-in-pcb"
 				(path "/204e071a-14ed-47a0-be54-332ac2b951cf/e7be5fc3-f0fe-4302-b3d4-c1d51cfac7bc"
-					(reference "J5")
+					(reference "XMOS_DEBUG1")
 					(unit 1)
 				)

Commit message: prepare for the 1st test batch
Parts:
- removed C53: 1uF, Capacitor_SMD:C_0402_1005Metric, symbol Device:C
- removed C54, C55: 20pF, Capacitor_SMD:C_0402_1005Metric, symbol Device:C
- removed FB4: 600R, Onju:BLM18PG121SN1D, symbol Device:FerriteBead
- removed R1, R2: 22R, Resistor_SMD:R_0402_1005Metric, symbol Seeed_libdb:Resistors/301010002
- removed R31: 680R, Resistor_SMD:R_0402_1005Metric, symbol Device:R
- removed R32: 1M, Resistor_SMD:R_0402_1005Metric, symbol Device:R
- removed U7: XU316-1024-QF60B-C24, Onju:XU316-1024-QF60B-C24, symbol New_Library:XU316-1024-QF60B-C24
- removed Y2: 24MHz, Crystal:Crystal_SMD_3225-4Pin_3.2x2.5mm, symbol Device:Crystal_GND24
- added C35, C39: 20pF, Capacitor_SMD:C_01005_0402Metric, symbol Seeed_libdb:Capacitors/302010050
- added C37: 1uF, Capacitor_SMD:C_01005_0402Metric, symbol Seeed_libdb:Capacitors/302013249
- added C44, C46, C47: 12pF, Capacitor:C0402, symbol Seeed_libdb:Capacitors/302010049
- added FB3: 600R, Inductor_SMD:L_0201_0603Metric, symbol Seeed_libadl:Ferrite Bead/303030521
- added R21: 1M, Resistor_SMD:R_01005_0402Metric, symbol Seeed_libadl:Resistors/301010009
- added R22: 680R, Resistor_SMD:R_01005_0402Metric, symbol Seeed_libadl:Resistors/301010505
- added R23, R24: 22R, Resistor_SMD:R_01005_0402Metric, symbol Seeed_libdb:Resistors/301010002
- added R25: 100R, Resistor_SMD:R_01005_0402Metric, symbol Seeed_libdb:Resistors/301010028
- added R26, R27, R28, R29, R30, R34, R36, R37, R38, R39: 0R, Resistor_SMD:R_01005_0402Metric, symbol Seeed_libdb:Resistors/301010000
- added R31: 10K, Resistor:R0402, symbol Seeed_libdb:Resistors/301010047
- added R32: 4.7K, Resistor:R0402, symbol Seeed_libdb:Resistors/301010010
- added R33: 330R, Resistor:R0402, symbol Seeed_libadl:Resistors/301010466
- added R35: 0R, Resistor_SMD:R_01005_0402Metric, symbol Seeed_libadl:Resistors/301010000
- added TP6, TP7, TP8: TEST-POINT, Seeed_Misc:TP-D45MIL, symbol 0_Seeed_Misc:TEST-POINT
- added TP9: Test Point, Misc:TP-D45MIL, symbol Seeed_libdb:Misc/TP45C_SMD
- added U7: XU316-1024-QF60B-C24​, Package_DFN_QFN:QFN-60-1EP_7x7mm_P0.4mm_EP3.4x3.4mm_ThermalVias, symbol reSpeaker:XU316-1024-QF60A-C24​
- added X1: 24MHz 12pF, Crystal:Crystal_SMD_2016-4Pin_2.0x1.6mm, symbol Seeed_libdb:OSC & XTAL/306011444
- XMOS_DEBUG1: now not fitted
- renumbered C37 to C36, C39 to C40, C40 to C41, C41 to C42, C42 to C43, C43 to C45, C142 to C48, C143 to C49, C44 to C50, C45 to C51, C46 to C52, C47 to C53, C48 to C54, C92 to C55, C49 to C56, C50 to C57, C51 to C58, C52 to C59, C59 to C60, C58 to C61, C56 to C62, C57 to C63, C60 to C64, C67 to C65, C68 to C66, C70 to C67, C69 to C68, D8 to D10, D5 to D11, D7 to D12, D3 to D6, D4 to D7, D2 to D8, D6 to D9, FB2 to FB4, FB3 to FB5, Q3 to Q2, Q2 to Q3, R29 to R40, R30 to R41, R63 to R42, R33 to R43, R34 to R44, R50 to R45, R4 to R46, R54 to R47, R53 to R48, R51 to R49, R6 to R50, R52 to R51, R5 to R52, R11 to R53, R12 to R54, R10 to R55, R13 to R56, R55 to R57, U9 to U10, U10 to U9
Connections:
- net +1V8: now also U7.17 (VDDIOB18), U7.26 (VDDIOB18), U7.31 (USB_VDD18)
- net +3V3: now also U7.30 (USB_VDD33)
- net GND: now also C35.2, C37.2, C39.2, C44.2, C46.2, C47.2, U7.65 (GND), X1.2, X1.4
- net I2C_SCL: now also U7.44 (X0D37)
- net I2C_SDA: now also U7.45 (X0D38)
- net I2S2_BCLK: now also R37.2
- net I2S2_DATA: now also R34.2
- net I2S2_LRCLK: now also U7.47 (X0D39)
- net I2S2_MCLK: now also R38.2
- net MIC_CLK: now also R25.2
- net MIC_DATA: now also U7.32 (X1D13)
- net QSPI_CLK: now also R33.2, U7.5 (X0D10)
- net QSPI_CS_N: now also U7.3 (X0D01)
- net QSPI_D0: now also U7.59 (X0D04)
- net QSPI_D1: now also R32.1, U7.1 (X0D05)
- net QSPI_D2: now also U7.60 (X0D06)
- net QSPI_D3: now also U7.2 (X0D07)
- net RST_N: now also U7.21 (RST_N)
- net TCK: now also U7.24 (TCK)
- net TDI: now also U7.18 (TDI)
- net TDO: now also U7.20 (TDO)
- net TMS: now also U7.23 (TMS)
- net VBUS_DETEC: now also U7.11 (X1D09)
- net VDD: now also FB3.2, U7.12 (VDD), U7.19 (VDD), U7.27 (VDD), U7.34 (VDD), U7.4 (VDD), U7.42 (VDD), U7.49 (VDD), U7.57 (VDD), U7.61 (VDD), U7.62 (VDD), U7.63 (VDD), U7.64 (VDD)
- net VDDIO: now also R31.2, U7.38 (VDDIOR), U7.52 (VDDIOT), U7.8 (VDDIOL)
- net XL_DN0: now also U7.35 (X1D17)
- net XL_DN1: now also U7.33 (X1D16)
- net XL_UP0: now also R23.2
- net XL_UP1: now also R24.2
- net XMOS_USB_N: now also U7.28 (USB_DM)
- net XMOS_USB_P: now also U7.29 (USB_DP)
- new net: R21.1, R22.1, U7.15 (XOUT)
- new net: C39.1, R22.2, X1.3
- new net: R23.1, U7.36 (X1D18)
- new net: R24.1, U7.37 (X1D19)
- new net: R28.1, U7.10 (X1D01)
- new net: R29.1, U7.13 (X1D10)
- new net: R30.1, U7.14 (X1D11)
- new net: C35.1, R21.2, U7.16 (XIN), X1.1
- new net: C37.1, FB3.1, U7.22 (PLL_AVDD)
- new net: R25.1, U7.39 (X1D22)
- new net: R37.1, U7.41 (X0D35)
- new net: R38.1, U7.43 (X0D36)
- new net: R26.1, U7.53 (X1D34)
- new net: R34.1, U7.7 (X0D11)
- new net: R27.1, U7.9 (X1D00)
- new net BOOT_SEL: R32.2, TP8.1 (T)
- new net BUT_A: U7.50 (X0D41)
- new net ESP_IO40: R39.2
- new net ESP_IO41: R36.2
- new net I2C2_SCL: U7.40 (X0D29)
- new net I2C2_SDA: U7.54 (X0D30)
- new net I2S_BCLK: C46.1, R29.2
- new net I2S_DIN_ESP: R26.2
- new net I2S_DIN_SEC: R27.2
- new net I2S_LRCK: C44.1, R28.2
- new net I2S_MCLK: C47.1, R30.2
- new net RST_DAC: R35.2
- new net SPI_CLK: R33.1, TP7.1 (T)
- new net SPI_CS_N: R31.1, TP6.1 (T), U7.6 (X0D00)
- new net XMOS_MUTE_DET: U7.46 (X0D40)
- new net XOD31: TP9.1 (T), U7.55 (X0D31)
- new net XOD32: R35.1, U7.56 (X0D32)
- new net XOD33: R36.1, U7.58 (X0D33)
- new net XOD43: R39.1, U7.51 (X0D43)
- new net XU316_WS2812: U7.48 (X0D42)
- no-connect marks 17 -> 2
Other:
- moved on the sheet: C36, C38, C40, C41, C42, C43, C45, C48, C49, C50, C51, C52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
