File: xmos.kicad_sch (KiCad schematic)
At the start: 96 parts, among them Q1 LBSS138WT1G, Q2 LBSS138WT1G, Q3 BC847B, U10 SN74LVC125APWR, U11 TLV73333PDBVR, U8 XU316-1024-QF60B-C24​, U9 W25Q32JVSSIQ, X1 24MHz 12pF

Commit message: prepare for the 1st test batch
Parts:
- added TP17: RST_N, TestPoint:TestPoint_Pad_D1.0mm, symbol Connector:TestPoint
- C42: footprint Capacitor_SMD:C_01005_0402Metric -> Capacitor_SMD:C_0402_1005Metric
- C49, C51, C52: footprint Capacitor:C0402 -> Capacitor_SMD:C_01005_0402Metric; Dielectric (none) -> NPO; Status Testo PoE -> (none); Voltage Rating 50V,NPO -> 50V
- R38: footprint Resistor:R0402 -> Resistor_SMD:R_01005_0402Metric; Power Rating 1% -> (none); Status Combox Pro -> (none); Tolerance (none) -> 1%
- R39, R40: Power Rating 5% -> (none); Status BeagleBone Carrier Board -> (none); Tolerance (none) -> 5%
- TP10: footprint Seeed_Misc:TP-D45MIL -> TestPoint:TestPoint_Pad_D1.0mm
- TP12: footprint Misc:TP-D45MIL -> TestPoint:TestPoint_Pad_D1.0mm
- X1: footprint Crystal:Crystal_SMD_2016-4Pin_2.0x1.6mm -> Onju:X4-SMD-2.0X1.6MM
Connections:
- net RST_N: now also TP17.1

Commit message: routing
Parts:
- C40, C44, C49, C51, C52: footprint Capacitor_SMD:C_01005_0402Metric -> Capacitor_SMD:C_0402_1005Metric
- C53, C54: Dielectric X5R -> X7R; Status BeagleBone Carrier Board -> (none); Voltage Rating 25V,X7R -> 25V
- R26, R27, R28, R29, R30, R31, R32, R33, R34, R35, R38, R39, R40, R41, R42, R43, R44: footprint Resistor_SMD:R_01005_0402Metric -> Resistor_SMD:R_0402_1005Metric
Changed lines of the file:
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@@
 			)
 		)
-		(property "Footprint" "Resistor_SMD:R_01005_0402Metric"
+		(property "Footprint" "Resistor_SMD:R_0402_1005Metric"
 			(at 66.04 149.86 0)
 			(effects
@@
 			)
 		)
-		(property "Footprint" "Resistor_SMD:R_01005_0402Metric"
+		(property "Footprint" "Resistor_SMD:R_0402_1005Metric"
 			(at 125.73 132.08 0)
 			(effects
@@
 			)
 		)
-		(property "Footprint" "Resistor_SMD:R_01005_0402Metric"
+		(property "Footprint" "Resistor_SMD:R_0402_1005Metric"
 			(at 125.73 134.62 0)
 			(effects
@@
 			)
 		)
-		(property "Footprint" "Resistor_SMD:R_01005_0402Metric"
+		(property "Footprint" "Resistor_SMD:R_0402_1005Metric"
 			(at 133.35 58.42 0)
 			(effects
@@
 			)
 		)
-		(property "Footprint" "Capacitor_SMD:C_01005_0402Metric"
+		(property "Footprint" "Capacitor_SMD:C_0402_1005Metric"
 			(at 166.37 123.19 0)
 			(effects
@@
 			)
 		)
-		(property "Footprint" "Resistor_SMD:R_01005_0402Metric"
+		(property "Footprint" "Resistor_SMD:R_0402_1005Metric"
 			(at 137.16 72.39 0)
 			(effects
@@
 			)
 		)
-		(property "Footprint" "Resistor_SMD:R_01005_0402Metric"
+		(property "Footprint" "Resistor_SMD:R_0402_1005Metric"
 			(at 130.81 106.68 0)
 			(effects
@@
 			)
 		)
-		(property "Footprint" "Resistor_SMD:R_01005_0402Metric"
+		(property "Footprint" "Resistor_SMD:R_0402_1005Metric"
 			(at 125.73 144.78 0)
 			(effects
@@
 			)
 		)
-		(property "Footprint" "Resistor_SMD:R_01005_0402Metric"
+		(property "Footprint" "Resistor_SMD:R_0402_1005Metric"
 			(at 133.35 60.96 0)
 			(effects
@@
 			)
 		)
-		(property "Footprint" "Resistor_SMD:R_01005_0402Metric"
+		(property "Footprint" "Resistor_SMD:R_0402_1005Metric"
 			(at 130.81 104.14 0)
 			(effects
@@
 			)
 		)
-		(property "Footprint" "Resistor_SMD:R_01005_0402Metric"
+		(property "Footprint" "Resistor_SMD:R_0402_1005Metric"
 			(at 130.81 116.84 0)
 			(effects
@@
 			)
 		)
-		(property "Footprint" "Resistor_SMD:R_01005_0402Metric"
+		(property "Footprint" "Resistor_SMD:R_0402_1005Metric"
 			(at 125.73 140.97 0)
 			(effects
@@
 			)
 		)
-		(property "Dielectric" "X5R"
-			(at 194.31 196.85 0)
+		(property "Dielectric" "X7R"
+			(at 198.12 201.168 0)
 			(effects
 				(font
@@
 			)
 		)
-		(property "Voltage Rating" "25V,X7R"
+		(property "Voltage Rating" "25V"
 			(at 196.215 199.39 0)
 			(effects
@@
 			)
 		)
-		(property "Status" "BeagleBone Carrier Board"
-			(at 194.31 196.85 0)
-			(effects
-				(font
-					(size 1.143 1.143)
-				)
-				(hide yes)
-			)
-		)
 		(property "Temperature" "-55°C to 125°C"
 			(at 194.31 196.85 0)
@@
 			)
 		)
-		(property "MANUFACTURER" ""
-			(at 194.31 196.85 0)
-			(effects
-				(font
-					(size 1.27 1.27)
-				)
-			)
-		)
-		(property "PARTREV" ""
-			(at 194.31 196.85 0)
-			(effects
-				(font
-					(size 1.27 1.27)
-				)
-			)
-		)
-		(property "STANDARD" ""
-			(at 194.31 196.85 0)
-			(effects
-				(font
-					(size 1.27 1.27)
-				)
-			)
-		)
 		(property "LCSC Part #" "C1525"
 			(at 194.31 196.85 0)
@@
 			)
 		)
-		(property "Dielectric" "X5R"
-			(at 194.31 223.52 0)
+		(property "Dielectric" "X7R"
+			(at 197.866 227.838 0)
 			(effects
 				(font
@@
 			)
 		)
-		(property "Voltage Rating" "25V,X7R"
+		(property "Voltage Rating" "25V"
 			(at 196.215 226.06 0)
 			(effects
@@
 			)
 		)
-		(property "Status" "BeagleBone Carrier Board"
-			(at 194.31 223.52 0)
-			(effects
-				(font
-					(size 1.143 1.143)
-				)
-				(hide yes)
-			)
-		)
 		(property "Temperature" "-55°C to 125°C"
 			(at 194.31 223.52 0)
@@
 			)
 		)
-		(property "MANUFACTURER" ""
-			(at 194.31 223.52 0)
-			(effects
-				(font
-					(size 1.27 1.27)
-				)
-			)
-		)
-		(property "PARTREV" ""
-			(at 194.31 223.52 0)
-			(effects
-				(font
-					(size 1.27 1.27)
-				)
-			)
-		)
-		(property "STANDARD" ""
-			(at 194.31 223.52 0)
-			(effects
-				(font
-					(size 1.27 1.27)
-				)
-			)
-		)
 		(property "LCSC Part #" "C1525"
 			(at 194.31 223.52 0)
@@
 			)
 		)
-		(property "Footprint" "Resistor_SMD:R_01005_0402Metric"
+		(property "Footprint" "Resistor_SMD:R_0402_1005Metric"
 			(at 137.16 99.06 0)
 			(effects
@@
 			)
 		)
-		(property "Footprint" "Resistor_SMD:R_01005_0402Metric"
+		(property "Footprint" "Resistor_SMD:R_0402_1005Metric"
 			(at 137.16 78.74 0)
 			(effects
@@
 			)
 		)
-		(property "Footprint" "Capacitor_SMD:C_01005_0402Metric"
+		(property "Footprint" "Capacitor_SMD:C_0402_1005Metric"
 			(at 175.26 123.19 0)
 			(effects
@@
 			)
 		)
-		(property "Footprint" "Capacitor_SMD:C_01005_0402Metric"
+		(property "Footprint" "Capacitor_SMD:C_0402_1005Metric"
 			(at 157.48 123.19 0)
 			(effects
@@
 			)
 		)
-		(property "Footprint" "Resistor_SMD:R_01005_0402Metric"
+		(property "Footprint" "Resistor_SMD:R_0402_1005Metric"
 			(at 50.8 143.51 0)
 			(effects
@@
 			)
 		)
-		(property "Footprint" "Capacitor_SMD:C_01005_0402Metric"
+		(property "Footprint" "Capacitor_SMD:C_0402_1005Metric"
 			(at 33.02 166.37 0)
 			(effects
@@
 			)
 		)
-		(property "Footprint" "Resistor_SMD:R_01005_0402Metric"
+		(property "Footprint" "Resistor_SMD:R_0402_1005Metric"
 			(at 137.16 74.93 0)
 			(effects
@@
 			)
 		)
-		(property "Footprint" "Resistor_SMD:R_01005_0402Metric"
+		(property "Footprint" "Resistor_SMD:R_0402_1005Metric"
 			(at 130.81 114.3 0)
 			(effects
@@
 			)
 		)
-		(property "Footprint" "Resistor_SMD:R_01005_0402Metric"
+		(property "Footprint" "Resistor_SMD:R_0402_1005Metric"
 			(at 137.16 81.28 0)
 			(effects
@@
 			)
 		)
-		(property "Footprint" "Capacitor_SMD:C_01005_0402Metric"
+		(property "Footprint" "Capacitor_SMD:C_0402_1005Metric"
 			(at 66.04 166.37 0)
 			(effects

Commit message: routing done
Parts:
- added R90: 0R, Resistor_SMD:R_0402_1005Metric, symbol Seeed_libdb:Resistors/301010000
Connections:
- net at U10.6 (2Y): now also R90.1; no longer D8.1
- net BUT_A: no longer names the net of U8.50 (X0D41)
- net XMOS_MUTE_DET: no longer names the net of U8.46 (X0D40)
- new net: D8.1, R90.2
- no-connect marks 2 -> 4
Other:
- moved on the sheet: C71, D8, R51, R55, R57, U10

Commit message: routing done
Parts:
- TP17: now not fitted

Commit message: ready for the 1st test batch
Parts:
- C40, C44: Dielectric (none) -> NP0; LCSC Part # (none) -> C1554; Manufacturer YAGEO -> FH (Guangdong Fenghua Advanced Tech); Manufacturer Part (none) -> 0402CG200J500NT; Voltage (none) -> 50V
- C42: Dielectric (none) -> X5R; LCSC Part # (none) -> C52923; Manufacturer Samsung -> Samsung Electro-Mechanics; Manufacturer Part (none) -> CL05A105KA5NQNC; Voltage (none) -> 25V
- C53, C54: Manufacturer YAGEO -> Samsung Electro-Mechanics; Manufacturer Part (none) -> CL05B104KO5NNNC; Voltage (none) -> 16V
- C60: Manufacturer YAGEO -> Samsung Electro-Mechanics; Manufacturer Part (none) -> CL05B104KO5NNNC
- C65: footprint Capacitor_SMD:C_0402_1005Metric -> Capacitor_SMD:C_0603_1608Metric
- FB3: footprint OPL_Filters_and_Magnetic_Beads:L0603 -> Onju:BLM18PG121SN1D; Current (none) -> 500mA; LCSC Part # (none) -> C85833; Manufacturer Part (none) -> BLM18KG601SN1D
- R26: LCSC Part # (none) -> C26083; Manufacturer YAGEO -> UNI-ROYAL(Uniroyal Elec); Manufacturer Part (none) -> 0402WGF1004TCE
- R27: LCSC Part # (none) -> C25130; Manufacturer YAGEO -> UNI-ROYAL(Uniroyal Elec); Manufacturer Part (none) -> 0402WGF6800TCE
- R28, R29: LCSC Part # (none) -> C25092; Manufacturer YAGEO -> UNI-ROYAL(Uniroyal Elec); Manufacturer Part (none) -> 0402WGF220JTCE
- R30: LCSC Part # (none) -> C25076; Manufacturer YAGEO -> UNI-ROYAL(Uniroyal Elec); Manufacturer Part (none) -> 0402WGF1000TCE
- R31, R32, R33, R34, R35, R39, R40, R41, R42, R43, R44, R90: LCSC Part # (none) -> C17168; Manufacturer YAGEO -> UNI-ROYAL(Uniroyal Elec); Manufacturer Part (none) -> 0402WGF0000TCE
- U8: LCSC Part # (none) -> C6617472; Manufacturer Part (none) -> XU316-1024-QF60B-C24
- U9: LCSC Part # (none) -> C179173; Manufacturer Part (none) -> W25Q32JVSSIQ
- X1: LCSC Part # (none) -> C252273; Manufacturer ECEC -> SJK(SHENZHEN CRYSTAL TECH); Manufacturer Part (none) -> 7F24000E12UCG

Commit message: final mods before production
Parts:
- removed D10, D11, D12, D6, D7, D9: PESD0402V05, Diode_SMD:D_0402_1005Metric, symbol Diode:SZESD9B5.0ST5G
