File: esp32.kicad_sch (KiCad schematic)
At the start: 36 parts, among them U5 ESP32-S3R8, U6 W25Q128JVSIQ, Y1 40MHz

Commit message: routing
Parts:
- removed R16: 499R, Resistor_SMD:R_0402_1005Metric, symbol Device:R
- removed R17: 0R, Resistor_SMD:R_0402_1005Metric, symbol Device:R
- removed R27, R28: 4.7k, Resistor_SMD:R_0402_1005Metric, symbol Device:R
- added SW2: BOOT, Onju:SW-SMD_4P-L4.2-W3.2-P2.15-LS4.5, symbol Switch:SW_Push
- added TP1: TOUCH_L, TestPoint:TestPoint_Pad_2.5x2.5mm, symbol Connector:TestPoint
- added TP2: TOUCH_C, TestPoint:TestPoint_Pad_2.5x2.5mm, symbol Connector:TestPoint
- added TP3: TOUCH_R, TestPoint:TestPoint_Pad_2.5x2.5mm, symbol Connector:TestPoint
- C28: LCSC Part # (none) -> C52923; Manufacturer (none) -> Samsung Electro-Mechanics; Manufacturer Part (none) -> CL05A105KA5NQNC; Supplier Part (none) -> C52923; Voltage 10V -> 25V
- C29: Dielectric NP0 -> C0G; LCSC Part # (none) -> C1547; Manufacturer (none) -> FH (Guangdong Fenghua Advanced Tech); Manufacturer Part (none) -> 0402CG120J500NT; Supplier Part (none) -> C1547
- D1: LCSC Part # (none) -> C83680; MANUFACTURER (none) -> LRC; MP (none) -> LRB520S-30T1G; Manufacturer (none) -> LRC; Manufacturer Part (none) -> LRB520S-30T1G; Supplier Part (none) -> C83680
- R23, R24: LCSC Part # (none) -> C25744; Manufacturer (none) -> UNI-ROYAL(Uniroyal Elec); Manufacturer Part (none) -> 0402WGF1002TCE; Supplier Part (none) -> C25744
Connections:
- net ESP_BOOT: now also SW2.1
- net GND: now also SW2.2
- net at C26.2, Y1.1: now also U5.53 (XTAL_N)
- net ECO_A: no longer names the net of U5.22 (XTAL_32K_N)
- net ECO_B: no longer names the net of U5.24 (GPIO18)
- net ESP_IO40: no longer names the net of U5.45 (MTDO)
- net ESP_IO41: no longer names the net of U5.47 (MTDI)
- net ESP_IO42: no longer names the net of U5.48 (MTMS)
- net ESP_IO48: no longer names the net of U5.36 (SPICLK_N)
- net ESP_RX0: no longer names the net of U5.50 (U0RXD)
- net I2C2_SCL: no longer names the net of U5.44 (MTCK)
- net I2C2_SDA: no longer names the net of U5.43 (GPIO38)
- net TOUCH_C: no longer names the net of U5.8 (GPIO3)
- net TOUCH_C: now also TP2.1
- net TOUCH_L: no longer names the net of U5.7 (GPIO2)
- net TOUCH_L: now also TP1.1
- net TOUCH_R: no longer names the net of U5.9 (GPIO4)
- net TOUCH_R: now also TP3.1
- no-connect marks 8 -> 18
Other:
- moved on the sheet: C28, C29, D1, R23, R24

Commit message: getting ready for production
Connections:
- net I2S_DIN_SEC is gone; now on net I2S2_DATA: U5.15 (GPIO10)
- net AUDIO_PA_EN: now also U5.24 (GPIO18); no longer U5.37 (SPICLK_P)
- net I2S2_DATA: no longer U5.21 (XTAL_32K_P)
- no-connect marks 18 -> 19

Commit message: getting ready for production
Parts:
- AE1: LCSC Part # (none) -> C89334; Manufacturer (none) -> JOHANSON DESIGN; Manufacturer Part (none) -> 2450AT18A100E
- C13: LCSC Part # (none) -> C327292; Manufacturer (none) -> YAGEO; Manufacturer Part (none) -> CC0402BRNPO9BN1R2; Voltage (none) -> 10V
Changed lines of the file:
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@@
+			)
+		)
+		(property "Voltage" "10V"
+			(at 64.77 71.12 90)
+			(effects
+				(font
+					(size 1.27 1.27)
+				)
+				(hide yes)
+			)
+		)
+		(property "LCSC Part #" "C327292"
+			(at 64.77 71.12 90)
+			(effects
+				(font
+					(size 1.27 1.27)
+				)
+				(hide yes)
+			)
+		)
+		(property "Manufacturer" "YAGEO"
+			(at 64.77 71.12 90)
+			(effects
+				(font
+					(size 1.27 1.27)
+				)
+				(hide yes)
+			)
+		)
+		(property "Manufacturer Part" "CC0402BRNPO9BN1R2"
+			(at 64.77 71.12 90)
+			(effects
+				(font
+					(size 1.27 1.27)
+				)
+				(hide yes)
 			)
 		)
@@
 			(at 29.21 66.04 0)
 			(effects
+				(font
+					(size 1.27 1.27)
+				)
+				(hide yes)
+			)
+		)
+		(property "LCSC Part #" "C89334"
+			(at 29.21 66.04 0)
+			(effects
+				(font
+					(size 1.27 1.27)
+				)
+				(hide yes)
+			)
+		)
+		(property "Manufacturer" "JOHANSON DESIGN"
+			(at 29.21 66.04 0)
+			(effects
+				(font
+					(size 1.27 1.27)
+				)
+				(hide yes)
+			)
+		)
+		(property "Manufacturer Part" "2450AT18A100E"
+			(at 29.21 66.04 0)
+			(effects

Commit message: update for production
Parts:
- C14: LCSC Part # (none) -> C48346; Manufacturer (none) -> FH (Guangdong Fenghua Advanced Tech); Manufacturer Part (none) -> 0402CG2R4C500NT
- C15, C16, C19, C20, C21, C23, C30: LCSC Part # (none) -> C1525; Manufacturer (none) -> Samsung Electro-Mechanics; Manufacturer Part (none) -> CL05B104KO5NNNC; Voltage 25V -> 16V
- C17, C22, C24: LCSC Part # (none) -> C52923; Manufacturer (none) -> Samsung Electro-Mechanics; Manufacturer Part (none) -> CL05A105KA5NQNC; Voltage 10V -> 25V
- C18: LCSC Part # (none) -> C15525; Manufacturer (none) -> Samsung Electro-Mechanics; Manufacturer Part (none) -> CL05A106MQ5NUNC; Voltage 10V -> 6.3V
- C25: LCSC Part # (none) -> C14663; Manufacturer (none) -> YAGEO; Manufacturer Part (none) -> CC0603KRX7R9BB104; Voltage 25V -> 50V
- C26, C27: LCSC Part # (none) -> C1547; Manufacturer (none) -> FH (Guangdong Fenghua Advanced Tech); Manufacturer Part (none) -> 0402CG120J500NT
- FB1: LCSC Part # (none) -> C14709; Manufacturer Part (none) -> BLM18PG121SN1D
- L2: LCSC Part # (none) -> C27124; Manufacturer (none) -> Sunlord; Manufacturer Part (none) -> SDCL1005C3N3STDF
- L4: LCSC Part # (none) -> C434826; Manufacturer (none) -> TDK; Manufacturer Part (none) -> MHQ1005P2N7BT000
- L5: LCSC Part # (none) -> C162540; Manufacturer (none) -> Murata Electronics; Manufacturer Part (none) -> LQG15HS2N2B02D
- R15: LCSC Part # (none) -> C17168; Manufacturer (none) -> UNI-ROYAL(Uniroyal Elec); Manufacturer Part (none) -> 0402WGF0000TCE
- R25, R26: LCSC Part # (none) -> C25900; Manufacturer (none) -> UNI-ROYAL(Uniroyal Elec); Manufacturer Part (none) -> 0402WGF4701TCE
- U5: LCSC Part # (none) -> C2913194; Manufacturer (none) -> Espressif Systems; Manufacturer Part (none) -> ESP32-S3R8
- U6: LCSC Part # (none) -> C97521; Manufacturer (none) -> Winbond Elec; Manufacturer Part (none) -> W25Q128JVSIQ
- Y1: LCSC Part # (none) -> C9010; Manufacturer (none) -> YXC Crystal Oscillators; Manufacturer Part (none) -> X322540MPB4SI
Connections:
- net ESP_RST renamed RST_BTN

Commit message: prepare for the 1st test batch
Parts:
- renumbered C25 to C17, C28 to C18, C27 to C19, C26 to C20, C13 to C21, C29 to C22, C19 to C23, C23 to C25, C20 to C26, C21 to C27, C22 to C28, C14 to C29, C15 to C30, C16 to C31, C17 to C32, C18 to C33, C30 to C34, D1 to D5, FB1 to FB2, L2 to L3, R23 to R16, R24 to R17, R15 to R18, R25 to R19, R26 to R20, TP1 to TP3, TP2 to TP4, TP3 to TP5

Commit message: prepare for the 1st test batch
Parts:
- renumbered C17 to C22, C18 to C23, C19 to C24, C20 to C25, C21 to C26, C22 to C27, C23 to C28, C24 to C29, C25 to C30, C26 to C31, C27 to C32, C28 to C33, C29 to C34, C30 to C35, C31 to C36, C32 to C37, C33 to C38, C34 to C39, R16 to R21, R17 to R22, R18 to R23, R19 to R24, R20 to R25, TP3 to TP6, TP4 to TP7, TP5 to TP8, U5 to U6, U6 to U7

Commit message: routing
Parts:
- added R82, R83, R84, R85, R86, R87, R88, R89: 0R, Resistor_SMD:R_0402_1005Metric, symbol Device:R
- added R90: 499R, Resistor_SMD:R_0402_1005Metric, symbol Device:R
Connections:
- net I2S2_BCLK: now also R88.2; no longer U6.18 (GPIO13)
- net I2S2_DATA: now also R85.2; no longer U6.15 (GPIO10)
- net I2S2_LRCLK: now also R89.2; no longer U6.19 (GPIO14)
- net I2S2_MCLK: now also R87.2; no longer U6.17 (GPIO12)
- net I2S_BCLK: now also R83.2; no longer U6.13 (GPIO8)
- net I2S_DIN_ESP: now also R86.2; no longer U6.16 (GPIO11)
- net I2S_LRCK: now also R82.2; no longer U6.12 (GPIO7)
- net I2S_MCLK: now also R84.2; no longer U6.14 (GPIO9)
- net XU316_RST: now also U6.52 (GPIO46); no longer U6.51 (GPIO45)
- net ESP_IO48: now reaches U6.36 (SPICLK_N)
- net I2C2_SCL: now reaches U6.44 (MTCK)
- net ESP_IIO40: now reaches U6.45 (MTDO)
- net ESP_IO41: now reaches U6.47 (MTDI)
- net ESP_IO42: now reaches U6.48 (MTMS)
- net at U6.49 (U0TXD): now also R90.2
- net ESP_RX0: now reaches U6.50 (U0RXD)
- new net: R83.1, U6.13 (GPIO8)
- new net: R89.1, U6.19 (GPIO14)
- new net: R82.1, U6.12 (GPIO7)
- new net: R84.1, U6.14 (GPIO9)
- new net: R85.1, U6.15 (GPIO10)
- new net: R86.1, U6.16 (GPIO11)
- new net: R87.1, U6.17 (GPIO12)
- new net: R88.1, U6.18 (GPIO13)
- new net ESP_TX0: R90.1
- new net WS2812_PWR: U6.51 (GPIO45)
- no-connect marks 19 -> 11

Commit message: routing
Parts:
- Y1: footprint Crystal:Crystal_SMD_3225-4Pin_3.2x2.5mm -> Crystal:Crystal_SMD_2016-4Pin_2.0x1.6mm; LCSC Part # C9010 -> (none); Manufacturer YXC Crystal Oscillators -> Murata; Manufacturer Part X322540MPB4SI -> XRCGB40M000F1S2SR0
Changed lines of the file:
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@@
 			)
 		)
-		(property "Footprint" "Crystal:Crystal_SMD_3225-4Pin_3.2x2.5mm"
+		(property "Footprint" "Crystal:Crystal_SMD_2016-4Pin_2.0x1.6mm"
 			(at 64.77 85.09 0)
 			(effects
@@
 			)
 		)
-		(property "Datasheet" "~"
+		(property "Datasheet" ""
 			(at 64.77 85.09 0)
 			(effects
@@
 			)
 		)
-		(property "Description" "±10ppm, 18pF, 50Ω, ABM8G-40.000MHZ-B2-T"
+		(property "Description" "40 MHz ±10ppm Crystal 9pF 50 Ohms 4-SMD, No Lead"
 			(at 64.77 85.09 0)
 			(effects
@@
 			)
 		)
-		(property "LCSC Part #" "C9010"
+		(property "LCSC Part #" ""
 			(at 64.77 85.09 90)
 			(effects
@@
 			)
 		)
-		(property "Manufacturer" "YXC Crystal Oscillators"
+		(property "Manufacturer" "Murata"
 			(at 64.77 85.09 90)
 			(effects
@@
 			)
 		)
-		(property "Manufacturer Part" "X322540MPB4SI"
+		(property "Manufacturer Part" "XRCGB40M000F1S2SR0"
 			(at 64.77 85.09 90)
 			(effects
