File: esp32.kicad_sch (KiCad schematic)
At the start: 45 parts, among them SW2 BOOT, U6 ESP32-S3R8, U7 W25Q128JVSIQ, Y1 40MHz

Commit message: routing done
Parts:
- removed R90: 499R, Resistor_SMD:R_0402_1005Metric, symbol Device:R
- added R91: 0R, Resistor_SMD:R_0402_1005Metric, symbol Device:R
Connections:
- net ESP_MUTE_DET: now also U6.6 (GPIO1); no longer U6.23 (GPIO17)
- net I2S2_DATA: now also R91.1; no longer R85.2
- net at U6.21 (XTAL_32K_P): now also R91.2
- net I2C2_SDA: now reaches U6.43 (GPIO38)
- net ESP_RX0: no longer names the net of U6.50 (U0RXD)
- net WS2812_PWR: no longer names the net of U6.51 (GPIO45)
- new net Audio_DET: U6.23 (GPIO17)
- new net I2S_DIN_SEC: R85.2

Commit message: routing done
Connections:
- net ESP_IIO40 renamed ESP_IO40

Commit message: ready for the 1st test batch
Parts:
- C27: Dielectric C0G -> NP0
- L3: LCSC Part # C27124 -> C16526
- R82, R83, R84, R85, R86, R87, R88, R89, R91: LCSC Part # (none) -> C17168; Manufacturer (none) -> UNI-ROYAL(Uniroyal Elec); Manufacturer Part (none) -> 0402WGF0000TCE
- Y1: LCSC Part # (none) -> C424431; Manufacturer Murata -> Yajingxin; Manufacturer Part XRCGB40M000F1S2SR0 -> TAXM40M4ZCBCDT2T

Commit message: mods after 1st batch testing
Connections:
- net Audio_DET: no longer names the net of U6.23 (GPIO17)
- no-connect marks 11 -> 12
Changed lines of the file:
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@@
+	)
+	(no_connect
+		(at 162.56 104.14)
 	)
 	(no_connect
@@
 		(pts
 			(xy 181.61 88.9) (xy 187.96 88.9)
-		)
-		(stroke
-			(width 0)
-			(type default)
-		)
-	)
-	(wire
-		(pts
-			(xy 187.96 104.14) (xy 162.56 104.14)
 		)
 		(stroke
@@
 			(effects
 				(font
-					(size 1.27 1.27)
-				)
-				(justify left)
-				(hide yes)
-			)
-		)
-	)
-	(global_label "Audio_DET"
-		(shape input)
-		(at 187.96 104.14 0)
-		(fields_autoplaced yes)
-		(effects
-			(font
-				(size 1.27 1.27)
-			)
-			(justify left)
-		)
-		(property "Intersheetrefs" "${INTERSHEET_REFS}"
-			(at 200.4398 104.14 0)
-			(effects
-				(font
