File: audio.kicad_sch (KiCad schematic)
At the start: 8 parts, among them J1 1775443-2, U11 MAX98357AETE_T

Commit message: update for production
Parts:
- C71, C72: LCSC Part # (none) -> C1710
- C73: LCSC Part # (none) -> C49678; Manufacturer (none) -> YAGEO; Manufacturer Part (none) -> CC0805KRX7R9BB104
- FB5, FB6: LCSC Part # (none) -> C85833; Manufacturer Part (none) -> BLM18KG601SN1D
- J1: LCSC Part # (none) -> C5162845; Manufacturer (none) -> TE Connectivity; Manufacturer Part (none) -> 1775443-2
- U11: LCSC Part # (none) -> C910544; Manufacturer (none) -> Analog Devices Inc./Maxim Integrated; Manufacturer Part (none) -> MAX98357AETE+T
Changed lines of the file:
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@@
+			)
+		)
+		(property "LCSC Part #" "C5162845"
+			(at 196.85 80.01 0)
+			(effects
+				(font
+					(size 1.27 1.27)
+				)
+				(hide yes)
+			)
+		)
+		(property "Manufacturer" "TE Connectivity"
+			(at 196.85 80.01 0)
+			(effects
+				(font
+					(size 1.27 1.27)
+				)
+				(hide yes)
+			)
+		)
+		(property "Manufacturer Part" "1775443-2"
+			(at 196.85 80.01 0)
+			(effects
+				(font
+					(size 1.27 1.27)
+				)
+				(hide yes)
 			)
 		)
@@
 		)
 		(property "Manufacturer" "Murata"
+			(at 170.18 77.47 90)
+			(effects
+				(font
+					(size 1.27 1.27)
+				)
+				(hide yes)
+			)
+		)
+		(property "LCSC Part #" "C85833"
+			(at 170.18 77.47 90)
+			(effects
+				(font
+					(size 1.27 1.27)
+				)
+				(hide yes)
+			)
+		)
+		(property "Manufacturer Part" "BLM18KG601SN1D"
 			(at 170.18 77.47 90)
 			(effects
@@
 			)
 		)
+		(property "LCSC Part #" "C49678"
+			(at 173.99 62.23 0)
+			(effects
+				(font
+					(size 1.27 1.27)
+				)
+				(hide yes)
+			)
+		)
+		(property "Manufacturer" "YAGEO"
+			(at 173.99 62.23 0)
+			(effects
+				(font
+					(size 1.27 1.27)
+				)
+				(hide yes)
+			)
+		)
+		(property "Manufacturer Part" "CC0805KRX7R9BB104"
+			(at 173.99 62.23 0)
+			(effects
+				(font
+					(size 1.27 1.27)
+				)
+				(hide yes)
+			)
+		)
 		(pin "1"
 		)
@@
 			)
 		)
+		(property "LCSC Part #" "C1710"
+			(at 189.23 90.17 0)
+			(effects
+				(font
+					(size 1.27 1.27)
+				)
+				(hide yes)
+			)
+		)
 		(pin "1"
 		)
@@
 		)
 		(property "Manufacturer" "Murata"
+			(at 170.18 85.09 90)
+			(effects
+				(font
+					(size 1.27 1.27)
+				)
+				(hide yes)
+			)
+		)
+		(property "LCSC Part #" "C85833"
+			(at 170.18 85.09 90)
+			(effects
+				(font
+					(size 1.27 1.27)
+				)
+				(hide yes)
+			)
+		)
+		(property "Manufacturer Part" "BLM18KG601SN1D"
 			(at 170.18 85.09 90)
 			(effects
@@
 			)
 		)
+		(property "LCSC Part #" "C910544"
+			(at 132.08 87.63 0)
+			(effects
+				(font
+					(size 1.27 1.27)
+				)
+				(hide yes)
+			)
+		)
+		(property "Manufacturer" "Analog Devices Inc./Maxim Integrated"
+			(at 132.08 87.63 0)
+			(effects
+				(font
+					(size 1.27 1.27)
+				)
+				(hide yes)
+			)
+		)
+		(property "Manufacturer Part" "MAX98357AETE+T"
+			(at 132.08 87.63 0)
+			(effects
+				(font
+					(size 1.27 1.27)
+				)
+				(hide yes)
+			)
+		)
 		(pin "7"
 		)
@@
 			(at 181.61 90.17 0)
 			(effects
+				(font
+					(size 1.27 1.27)
+				)
+				(hide yes)
+			)
+		)
+		(property "LCSC Part #" "C1710"
+			(at 181.61 90.17 0)
+			(effects

Commit message: prepare for the 1st test batch
Parts:
- removed C71, C72: 10nF, Capacitor_SMD:C_0805_2012Metric, symbol Device:C
- removed C73: 100nF, Capacitor_SMD:C_0805_2012Metric, symbol Device:C
- removed C74: 47uF, Capacitor_SMD:C_0805_2012Metric, symbol Device:C
- removed FB5, FB6: 600R, Onju:BLM18PG121SN1D, symbol Device:FerriteBead
- removed J1: 1775443-2, Onju:1775443-2, symbol New_Library:1775443-2
- removed U11: MAX98357AETE_T, Onju:max98357aete, symbol New_Library:MAX98357AETE_T
- added C69: 2.2uF, Capacitor:C0603, symbol Seeed_libdb:Capacitors/302010054
- added C70, C72, C74, C76, C77, C78, C79, C81, C82, C83: 100nF, Capacitor:C0402, symbol Seeed_libadl:Capacitors/302010024
- added C71, C84, C86: 10uF, Capacitor:C0603, symbol Seeed_libdb:Capacitors/302013252
- added C73, C80, C87: 1uF, Capacitor:C0402, symbol Seeed_libdb:Capacitors/302013249
- added C75, C85: 22uF, Capacitor:C0603, symbol Seeed_libdb:Capacitors/302013254
- added C88, C89: 4.7nF, Capacitor:C0402, symbol Seeed_libdb:Capacitors/302010261
- added C90, C91, C92: 22uF, Capacitor:C0805, symbol Seeed_libdb:Capacitors/302013260
- added C93: 10nF, Capacitor:C0402, symbol Seeed_libadl:Capacitors/302010006
- added C94, C96: 100nF, Capacitor:C0603, symbol Seeed_libdb:Capacitors/302010138
- added C95: 47uF, Capacitor:C1206, symbol Seeed_libdb:Capacitors/302013265
- added C97, C98: 10nF, Capacitor:C0402, symbol Seeed_libdb:Capacitors/302010006
- added D13: LRB520S-30T1G, Diode:SOD-523, symbol Seeed_libdb:Diode/304011072
- added FB6: 120R, Inductor:L0603, symbol Seeed_libadl:Ferrite Bead/303030024
- added FB7, FB8: 600R, Inductor:L0603, symbol Seeed_libdb:Ferrite Bead/303030521
- added J2: WY-3315, Connector:JST2P_1d25_7_55x4_25x4_8mm, symbol Seeed_libdb:Connector/320111167
- added Q4: LBSS138WT1G, Mosfet:SOT-323, symbol Seeed_libadl:Mosfet/305031542
- added R58, R59: 0R, Resistor:R0805, symbol Seeed_libdb:Resistors/301010359
- added R60, R61, R64, R65: 10K, Resistor:R0402, symbol Seeed_libadl:Resistors/301010047
- added R62, R63: 0R, Resistor:R0402, symbol Seeed_libdb:Resistors/301010000
- added R66, R67, R68, R76: 0R, Resistor:R0603, symbol Seeed_libdb:Resistors/301010292
- added R69, R70: 0R, Resistor:R0402, symbol Seeed_libadl:Resistors/301010000
- added R71: 4.7K, Resistor:R0402, symbol Seeed_libdb:Resistors/301010010
- added R72: 470K, Resistor:R0402, symbol Seeed_libdb:Resistors/301010069
- added R73, R74, R75: 15K, Resistor:R0603, symbol Seeed_libdb:Resistors/301010241
- added TP10, TP12: TEST-POINT, Seeed_Misc:TP-D45MIL, symbol 0_Seeed_Misc:TEST-POINT
- added TP11, TP13: Test Point, Misc:TP-D45MIL, symbol libdb:Misc/TP45C_SMD
- added U11: LC1458CB5TR33, Ic:SOT-23-5, symbol Seeed_libdb:Ic/310032530
- added U12: TLV320AIC3204IRHBR, reSpeaker Library:TLV320AIC3204IRHBR, symbol reSpeaker:TLV320AIC3204IRHBR
- added U13: TPA6211A1DGNR, Ic:DGN8_1d89X1P57, symbol Seeed_libdb:Ic/TPA6211A1DGNR
Connections:
- net +5V: now also C69.1, C70.1, R76.1, U11.1 (IN)
- net AUDIO_PA_EN: now also R69.1
- net GND: now also C69.2, C70.2, C71.2, C72.2, C73.2, C74.2, C75.2, C76.2, C78.2, C80.2, C84.2, C93.2, Q4.2 (S), R58.1, R59.1, R64.1, R72.1, U11.2 (GND), U12.28 (DVSS), U12.33 (EP), U12.7 (IOVSS)
- net I2S_BCLK: now also U12.2 (BCLK)
- net I2S_DIN_ESP: now also U12.4 (DIN_/_MFP1)
- net I2S_LRCK: now also U12.3 (WCLK)
- new net: C75.1, C76.1, U12.29 (DVDD)
- new net: C91.2, R74.1
- new net: R74.2, R75.2, U13.4 (IN-)
- new net: C94.2, U13.2 (BYPASS)
- new net: R73.2, U13.3 (IN+)
- new net: FB8.1, U13.5 (VO+)
- new net: FB7.1, U13.8 (VO-)
- new net: C81.1, C85.1, U12.24 (AVDD)
- new net: R63.2, U12.10 (SDA/MOSI)
- new net: R64.2, U12.12 (SPI__SELECT)
- new net: C77.1, U12.13 (IN1_L), U12.14 (IN1_R)
- new net: C79.1, U12.15 (IN2_L), U12.16 (IN2_R)
- new net: C82.1, C86.1, C87.1, U12.18 (REF)
- new net: C83.1, U12.20 (IN3_L), U12.21 (IN3_R)
- new net: R68.1, U12.22 (LOL)
- new net: R67.1, U12.23 (LOR)
- new net: R61.1, U12.30 (LDO__SELECT)
- new net: R62.2, U12.9 (SCL/~{SS})
- new net: C88.1, C91.1, R67.2
- new net: R69.2, R70.2, R71.2
- new net: C90.2, R73.1
- new net: C89.1, C92.1, R68.2
- new net: C92.2, R75.1
- new net +3.3VA: C71.1, C72.1, C73.1, C74.1, C78.1, C80.1, C84.1, FB6.2, R60.2, R61.2, TP11.1 (T), U11.5 (OUT), U12.26 (LDOIN), U12.6 (IOVDD)
- new net +3V3: FB6.1, R65.2, R70.1, U11.3 (EN)
- new net AMP_CTL: C93.1, Q4.3 (D), R71.1, R72.2, TP12.1 (T), U13.1 (*SHUTDOWN)
- new net Audio_DET: D13.1, Q4.1 (G), R65.1
- new net GNDA: C77.2, C79.2, C81.2, C82.2, C83.2, C85.2, C86.2, C87.2, C88.2, C89.2, C90.1, C94.1, C95.2, C96.2, C97.2, C98.2, J2.3, J2.4, R58.2, R59.2, R66.2, U12.17 (AVSS), U13.7 (GND), U13.EPAD
- new net I2C_SCL: R62.1
- new net I2C_SDA: R63.1
- new net I2S_DIN_SEC: U12.8 (SCLK_/_MFP3)
- new net I2S_MCLK: U12.1 (MCLK)
- new net MICDET: D13.2, R66.1
- new net PA_5V: C95.1, C96.1, R76.2, TP13.1 (T), U13.6 (VDD)
- new net RST_DAC: R60.1, TP10.1 (T), U12.31 (~{RESET})
- new net SKP-: C98.1, FB7.2, J2.2
- new net SPK+: C97.1, FB8.2, J2.1
- no-connect marks 1 -> 7
Other:
- note added: "I2C Addr: 0X18"

Commit message: prepare for the 1st test batch
Parts:
- removed J2: WY-3315, Connector:JST2P_1d25_7_55x4_25x4_8mm, symbol Seeed_libdb:Connector/320111167
- added J2: 1775443-2, Onju:1775443-2, symbol New_Library:1775443-2
- renumbered C95 to C100, C96 to C101, C97 to C102, C98 to C103, C69 to C74, C70 to C75, C71 to C76, C72 to C77, C73 to C78, C74 to C79, C75 to C80, C76 to C81, C77 to C82, C78 to C83, C79 to C84, C80 to C85, C81 to C86, C82 to C87, C83 to C88, C84 to C89, C85 to C90, C86 to C91, C87 to C92, C88 to C93, C89 to C94, C90 to C95, C91 to C96, C92 to C97, C93 to C98, C94 to C99, R58 to R63, R59 to R64, R60 to R65, R61 to R66, R62 to R67, R63 to R68, R64 to R69, R65 to R70, R66 to R71, R67 to R72, R68 to R73, R69 to R74, R70 to R75, R71 to R76, R72 to R77, R73 to R78, R74 to R79, R75 to R80, R76 to R81, TP10 to TP13, TP11 to TP14, TP12 to TP15, TP13 to TP16, U11 to U12, U12 to U13, U13 to U14
Connections:
- net SPK+: now also J2.2
- net SKP- renamed SPK-
- net SPK-: now also J2.1

Commit message: routing
Parts:
- removed FB6: 120R, Inductor:L0603, symbol Seeed_libadl:Ferrite Bead/303030024
- added FB9: 120R, Onju:BLM18PG121SN1D, symbol Device:FerriteBead
- C74: footprint Capacitor:C0603 -> Capacitor_SMD:C_0603_1608Metric; Dielectric (none) -> X7R; Voltage Rating 10V,X7R -> 10V
- C75, C79, C81, C83, C86, C88: footprint Capacitor:C0402 -> Capacitor_SMD:C_0402_1005Metric; Dielectric (none) -> X7R; Status BeagleBone Carrier Board -> (none); Voltage Rating 25V,X7R -> 25V
- C76, C89: footprint Capacitor:C0603 -> Capacitor_SMD:C_0603_1608Metric; Dielectric (none) -> X5R; Status HA VOICE KIT -> (none); Voltage Rating 10V,X5R -> 10V
- C78, C85: footprint Capacitor:C0402 -> Capacitor_SMD:C_0402_1005Metric; Dielectric (none) -> X5R; Status HA Voice KIT -> (none); Voltage Rating 10V,X5R -> 10V
- C80, C90: footprint Capacitor:C0603 -> Capacitor_SMD:C_0603_1608Metric; Dielectric (none) -> X5R; Status reSpeaker -> (none); Voltage Rating 6.3V,X5R -> 6.3V
- R65, R66: footprint Resistor:R0402 -> Resistor_SMD:R_0402_1005Metric; Part Type RES -> (none); Power Rating 1% -> (none); Status BeagleBone Carrier Board -> (none); Tolerance (none) -> 1%
- R71: footprint Resistor:R0603 -> Resistor_SMD:R_0603_1608Metric; Part Type RES -> (none); Power Rating 5% -> (none); Tolerance (none) -> 5%
- TP13: footprint Seeed_Misc:TP-D45MIL -> TestPoint:TestPoint_Pad_D1.0mm
- TP14: footprint Misc:TP-D45MIL -> TestPoint:TestPoint_Pad_D1.0mm; SKU TP45C_SMD -> (none)
Connections:
- net +3.3VA: now also FB9.2
- net +3V3: now also FB9.1

Commit message: routing
Parts:
- removed C74: 2.2uF, Capacitor_SMD:C_0603_1608Metric, symbol Seeed_libdb:Capacitors/302010054
- removed C75, C79: 100nF, Capacitor_SMD:C_0402_1005Metric, symbol Seeed_libadl:Capacitors/302010024
- removed C78: 1uF, Capacitor_SMD:C_0402_1005Metric, symbol Seeed_libdb:Capacitors/302013249
- removed C93, C94: 4.7nF, Capacitor:C0402, symbol Seeed_libdb:Capacitors/302010261
- removed R63, R64: 0R, Resistor:R0805, symbol Seeed_libdb:Resistors/301010359
- removed R72, R73: 0R, Resistor:R0603, symbol Seeed_libdb:Resistors/301010292
- removed U12: LC1458CB5TR33, Ic:SOT-23-5, symbol Seeed_libdb:Ic/310032530
- added R63, R64, R72, R73: 0R, Resistor_SMD:R_0402_1005Metric, symbol Seeed_libdb:Resistors/301010000
- C77, C82, C84, C87: footprint Capacitor:C0402 -> Capacitor_SMD:C_0402_1005Metric; Dielectric (none) -> X7R; Status BeagleBone Carrier Board -> (none); Voltage Rating 25V,X7R -> 25V
- C91: footprint Capacitor:C0603 -> Capacitor_SMD:C_0603_1608Metric; Dielectric (none) -> X5R; Status HA VOICE KIT -> (none); Voltage Rating 10V,X5R -> 10V
- C92: footprint Capacitor:C0402 -> Capacitor_SMD:C_0402_1005Metric; Dielectric (none) -> X5R; Status HA Voice KIT -> (none); Voltage Rating 10V,X5R -> 10V
- C95, C96, C97: footprint Capacitor:C0805 -> Capacitor_SMD:C_0805_2012Metric; Priority A -> (none)
- C99: footprint Capacitor:C0603 -> Capacitor_SMD:C_0603_1608Metric; Dielectric (none) -> X7R; Status BeagleBone Carrier Board -> (none); Voltage Rating 50V,X7R -> 50V
- R67, R68: footprint Resistor:R0402 -> Resistor_SMD:R_0402_1005Metric; Power Rating 5% -> (none); Status BeagleBone Carrier Board -> (none); Tolerance (none) -> 5%
- R69: footprint Resistor:R0402 -> Resistor_SMD:R_0402_1005Metric; Power Rating 1% -> (none); Status BeagleBone Carrier Board -> (none); Tolerance (none) -> 1%
- R78, R79, R80: footprint Resistor:R0603 -> Capacitor_SMD:C_0603_1608Metric; Power Rating 1% -> (none); Status Sensecap Gateway V1 -> (none); Tolerance (none) -> 1%
- U13: footprint reSpeaker Library:TLV320AIC3204IRHBR -> Onju:TLV320AIC3204IRHBR
- U14: footprint Ic:DGN8_1d89X1P57 -> Onju:TPA6211A1DGNR; Status HA Voice Kit -> (none)
Connections:
- net GND: now also R63.1, R64.1
- net GNDA: now also R63.2, R64.2
- net at R79.1: now also C97.2; no longer C96.2
- net at U13.22 (LOL): now also R73.1
- net at U13.23 (LOR): now also R72.1
- net at C96.1: now also R72.2
- net at C97.1: now also R73.2
- net at R80.1: now also C96.2; no longer C97.2
- no-connect marks 7 -> 6

Commit message: routing
Parts:
- C100: footprint Capacitor:C1206 -> Capacitor_SMD:C_1206_3216Metric; Dielectric (none) -> X5R; Status reSpeaker -> (none); Voltage Rating 10V,X5R -> 10V
- C101: footprint Capacitor:C0603 -> Capacitor_SMD:C_0603_1608Metric; Dielectric (none) -> X7R; Status BeagleBone Carrier Board -> (none); Voltage Rating 50V,X7R -> 50V
- C102, C103, C98: footprint Capacitor:C0402 -> Capacitor_SMD:C_0402_1005Metric; Dielectric (none) -> X7R; Status BeagleBone Carrier Board -> (none); Voltage Rating 50V,X7R -> 50V
- D13: footprint Diode:SOD-523 -> Diode_SMD:D_SOD-523
- FB7, FB8: footprint Inductor:L0603 -> Inductor_SMD:L_0603_1608Metric; Status ReCamera-Pre -> (none)
- Q4: footprint Mosfet:SOT-323 -> Package_TO_SOT_SMD:SOT-323_SC-70
- R70: footprint Resistor:R0402 -> Resistor_SMD:R_0402_1005Metric; Power Rating 1% -> (none); Status BeagleBone Carrier Board -> (none); Tolerance (none) -> 1%
- R74, R75, R76: footprint Resistor:R0402 -> Resistor_SMD:R_0402_1005Metric; Power Rating 5% -> (none); Status BeagleBone Carrier Board -> (none); Tolerance (none) -> 5%
- R77: footprint Resistor:R0402 -> Resistor_SMD:R_0402_1005Metric; Power Rating 1% -> (none); Status Combox Pro -> (none); Tolerance (none) -> 1%
- R81: footprint Resistor:R0603 -> Resistor_SMD:R_0603_1608Metric; Power Rating 5% -> (none); Tolerance (none) -> 5%
- TP15: footprint Seeed_Misc:TP-D45MIL -> TestPoint:TestPoint_Pad_D1.0mm
- TP16: footprint Misc:TP-D45MIL -> TestPoint:TestPoint_Pad_D1.0mm

Commit message: routing done
Parts:
- R78, R79, R80: footprint Capacitor_SMD:C_0603_1608Metric -> Resistor_SMD:R_0603_1608Metric

Commit message: ready for the 1st test batch
Parts:
- C100: LCSC Part # (none) -> C96123; Manufacturer Samsung -> Samsung Electro-Mechanics; Manufacturer Part (none) -> CL31A476MPHNNNE; Voltage (none) -> 10V
- C101, C99: LCSC Part # (none) -> C14663; Manufacturer Part (none) -> CC0603KRX7R9BB104; Voltage (none) -> 50V
- C102, C103, C98: LCSC Part # (none) -> C15195; Manufacturer YAGEO -> Samsung Electro-Mechanics; Manufacturer Part (none) -> CL05B103KB5NNNC; Voltage (none) -> 50V
- C76, C89, C91: LCSC Part # (none) -> C19702; Manufacturer Samsung -> Samsung Electro-Mechanics; Manufacturer Part (none) -> CL10A106KP8NNNC; Voltage (none) -> 10V
- C77, C81, C82, C83, C84, C86, C87, C88: LCSC Part # (none) -> C1525; Manufacturer YAGEO -> Samsung Electro-Mechanics; Manufacturer Part (none) -> CL05B104KO5NNNC; Voltage (none) -> 16V
- C80, C90: LCSC Part # (none) -> C59461; Manufacturer Samsung -> Samsung Electro-Mechanics; Manufacturer Part (none) -> CL10A226MQ8NRNC; Voltage (none) -> 6.3V
- C85, C92: LCSC Part # (none) -> C52923; Manufacturer Samsung -> Samsung Electro-Mechanics; Manufacturer Part (none) -> CL05A105KA5NQNC
- C95, C96, C97: LCSC Part # (none) -> C45783; Manufacturer Samsung -> Samsung Electro-Mechanics; Manufacturer Part (none) -> CL21A226MAQNNNE; Voltage (none) -> 25V
- D13: LCSC Part # (none) -> C83680; Manufacturer Part (none) -> LRB520S-30T1G
- FB7, FB8: Current (none) -> 500mA; LCSC Part # (none) -> C85833; Manufacturer Part (none) -> BLM18KG601SN1D
- Q4: LCSC Part # (none) -> C383201; Manufacturer Part (none) -> LBSS138WT1G
- R63, R64, R67, R68, R72, R73, R74: LCSC Part # (none) -> C17168; Manufacturer YAGEO -> UNI-ROYAL(Uniroyal Elec); Manufacturer Part (none) -> 0402WGF0000TCE
- R65, R66, R69, R70: LCSC Part # (none) -> C25744; Manufacturer YAGEO -> UNI-ROYAL(Uniroyal Elec); Manufacturer Part (none) -> 0402WGF1002TCE
- R71: LCSC Part # (none) -> C21189; MPN RC0603JR-070RL -> (none); Manufacturer YAGEO -> UNI-ROYAL(Uniroyal Elec); Manufacturer Part (none) -> 0603WAF0000T5E; SKU 301010292 -> (none)
- R76: LCSC Part # (none) -> C25900; Manufacturer YAGEO -> UNI-ROYAL(Uniroyal Elec); Manufacturer Part (none) -> 0402WGF4701TCE
- R77: LCSC Part # (none) -> C25790; MPN RC0402FR-07470KL -> (none); Manufacturer YAGEO -> UNI-ROYAL(Uniroyal Elec); Manufacturer Part (none) -> 0402WGF4703TCE; Part Type RES -> (none); SKU 301010069 -> (none)
- R78, R79, R80: LCSC Part # (none) -> C22809; MPN RC0603FR-0715KL -> (none); Manufacturer YAGEO -> UNI-ROYAL(Uniroyal Elec); Manufacturer Part (none) -> 0603WAF1502T5E; Part Type RES -> (none); SKU 301010241 -> (none)
- R81: LCSC Part # (none) -> C21189; MPN RC0603JR-070RL -> (none); Manufacturer YAGEO -> UNI-ROYAL(Uniroyal Elec); Manufacturer Part (none) -> 0603WAF0000T5E; Part Type RES -> (none); SKU 301010292 -> (none)
- U13: LCSC Part # (none) -> C24109; Manufacturer Part (none) -> TLV320AIC3204IRHBR
- U14: LCSC Part # (none) -> C7718; Manufacturer TI -> Texas Instruments; Manufacturer Part (none) -> TPA6211A1DGNR
