File: audio.kicad_sch (KiCad schematic)
At the start: 55 parts, among them J2 1775443-2, Q4 LBSS138WT1G, U13 TLV320AIC3204IRHBR, U14 TPA6211A1DGNR

Commit message: mods after 1st batch testing
Parts:
- removed D13: LRB520S-30T1G, Diode_SMD:D_SOD-523, symbol Seeed_libdb:Diode/304011072
- removed Q4: LBSS138WT1G, Package_TO_SOT_SMD:SOT-323_SC-70, symbol Seeed_libadl:Mosfet/305031542
- removed R70: 10K, Resistor_SMD:R_0402_1005Metric, symbol Seeed_libadl:Resistors/301010047
- removed R71: 0R, Resistor_SMD:R_0603_1608Metric, symbol Seeed_libdb:Resistors/301010292
