File: audio.kicad_sch (KiCad schematic)
At the start: 51 parts, among them J2 1775443-2, U13 TLV320AIC3204IRHBR, U14 TPA6211A1DGNR

Commit message: v2 hardware revision
MPR121 touch controller added to replace esp32-s3 integrated touch pins
Parts:
- removed R75: 0R, Resistor_SMD:R_0402_1005Metric, symbol Seeed_libadl:Resistors/301010000
- C100: Function (none) -> AUDIO; SKU 302013265 -> (none)
- C101, C99: Function (none) -> POWER; SKU 302010138 -> (none)
- C102, C103, C98: Function (none) -> AUDIO; SKU 302010006 -> (none)
- C76, C89, C91: Function (none) -> AUDIO; SKU 302013252 -> (none)
- C77, C81, C82, C83, C84, C86, C87, C88: Function (none) -> POWER; SKU 302010024 -> (none)
- C80, C90: Function (none) -> AUDIO; SKU 302013254 -> (none)
- C85, C92: Function (none) -> AUDIO; SKU 302013249 -> (none)
- C95, C96, C97: Function (none) -> POWER; SKU 302013260 -> (none)
- FB7, FB8: Function (none) -> AUDIO; SKU 303030521 -> (none)
- FB9: Part number BLM18PG121SN1D -> (none)
- J2: Availability In Stock -> (none); Centerline_Pitch 1.5 mm[.059 in] -> (none); Check_prices https://www.snapeda.com/parts/1775443-2/TE+Connectivity/vie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 -> (none); Comment 1775443-2 -> (none); EU_RoHS_Compliance Compliant -> (none); Number_of_Positions 2 -> (none); PARTREV B5 -> (none); Supplier Part C5162845 -> (none)
- R63, R64, R67, R68, R72, R73, R74: Function (none) -> AUDIO; SKU 301010000 -> (none)
- R65, R66, R69: Function (none) -> AUDIO; SKU 301010047 -> (none)
- R76: Function (none) -> AUDIO; SKU 301010010 -> (none)
- R77, R78, R79, R80, R81: Function (none) -> AUDIO
- TP16: SKU TP45C_SMD -> (none)
- U13: Arrow Part Number TLV320AIC3204IRHBR -> (none); Arrow Price/Stock https://www.arrow.com/en/products/tlv320aic3204irhbr/texas-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 -> (none); Function (none) -> AUDIO; Height 1 -> (none); Mouser Price/Stock https://www.mouser.co.uk/ProductDetail/Texas-Instruments/TL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 -> (none); SKU 310080252 -> (none)
- U14: Function (none) -> AUDIO; SKU 310020941 -> (none)
