File: leds.kicad_sch (KiCad schematic)
At the start: 8 parts

Commit message: routing
Connections:
- no-connect marks 0 -> 1
Changed lines of the file:
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@@
 		(color 0 0 0 0)
+	)
+	(no_connect
+		(at 219.71 76.2)
 	)
 	(wire

Commit message: update for production
Parts:
- C31, C32, C33, C34: LCSC Part # (none) -> C1525; Manufacturer (none) -> YAGEO; Voltage 10V -> 16V
- LED2, LED3, LED4, LED5: LCSC Part # (none) -> C5149201; Manufacturer (none) -> OPSCO Optoelectronics; Manufacturer Part (none) -> SK6812MINI-E
Changed lines of the file:
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@@
 			)
 		)
-		(property "Voltage" "10V"
+		(property "Voltage" "16V"
 			(at 107.188 78.994 0)
 			(effects
@@
 		)
 		(property "Function" "LED"
+			(at 102.87 76.2 0)
+			(effects
+				(font
+					(size 1.27 1.27)
+				)
+				(hide yes)
+			)
+		)
+		(property "LCSC Part #" "C1525"
+			(at 102.87 76.2 0)
+			(effects
+				(font
+					(size 1.27 1.27)
+				)
+				(hide yes)
+			)
+		)
+		(property "Manufacturer" "YAGEO"
 			(at 102.87 76.2 0)
 			(effects
@@
 			)
 		)
+		(property "LCSC Part #" "C5149201"
+			(at 85.09 76.2 0)
+			(effects
+				(font
+					(size 1.27 1.27)
+				)
+				(hide yes)
+			)
+		)
+		(property "Manufacturer" "OPSCO Optoelectronics"
+			(at 85.09 76.2 0)
+			(effects
+				(font
+					(size 1.27 1.27)
+				)
+				(hide yes)
+			)
+		)
+		(property "Manufacturer Part" "SK6812MINI-E"
+			(at 85.09 76.2 0)
+			(effects
+				(font
+					(size 1.27 1.27)
+				)
+				(hide yes)
+			)
+		)
 		(pin "2"
 		)
@@
 			)
 		)
+		(property "LCSC Part #" "C5149201"
+			(at 125.73 76.2 0)
+			(effects
+				(font
+					(size 1.27 1.27)
+				)
+				(hide yes)
+			)
+		)
+		(property "Manufacturer" "OPSCO Optoelectronics"
+			(at 125.73 76.2 0)
+			(effects
+				(font
+					(size 1.27 1.27)
+				)
+				(hide yes)
+			)
+		)
+		(property "Manufacturer Part" "SK6812MINI-E"
+			(at 125.73 76.2 0)
+			(effects
+				(font
+					(size 1.27 1.27)
+				)
+				(hide yes)
+			)
+		)
 		(pin "2"
 		)
@@
 			)
 		)
+		(property "LCSC Part #" "C5149201"
+			(at 165.1 76.2 0)
+			(effects
+				(font
+					(size 1.27 1.27)
+				)
+				(hide yes)
+			)
+		)
+		(property "Manufacturer" "OPSCO Optoelectronics"
+			(at 165.1 76.2 0)
+			(effects
+				(font
+					(size 1.27 1.27)
+				)
+				(hide yes)
+			)
+		)
+		(property "Manufacturer Part" "SK6812MINI-E"
+			(at 165.1 76.2 0)
+			(effects
+				(font
+					(size 1.27 1.27)
+				)
+				(hide yes)
+			)
+		)
 		(pin "2"
 		)
@@
 			)
 		)
-		(property "Voltage" "10V"
+		(property "Voltage" "16V"
 			(at 226.568 78.994 0)
 			(effects
@@
 		)
 		(property "Function" "LED"
+			(at 222.25 76.2 0)
+			(effects
+				(font
+					(size 1.27 1.27)
+				)
+				(hide yes)
+			)
+		)
+		(property "LCSC Part #" "C1525"
+			(at 222.25 76.2 0)
+			(effects
+				(font
+					(size 1.27 1.27)
+				)
+				(hide yes)
+			)
+		)
+		(property "Manufacturer" "YAGEO"
 			(at 222.25 76.2 0)
 			(effects
@@
 			)
 		)
+		(property "LCSC Part #" "C5149201"
+			(at 204.47 76.2 0)
+			(effects
+				(font
+					(size 1.27 1.27)
+				)
+				(hide yes)
+			)
+		)
+		(property "Manufacturer" "OPSCO Optoelectronics"
+			(at 204.47 76.2 0)
+			(effects
+				(font
+					(size 1.27 1.27)
+				)
+				(hide yes)
+			)
+		)
+		(property "Manufacturer Part" "SK6812MINI-E"
+			(at 204.47 76.2 0)
+			(effects
+				(font
+					(size 1.27 1.27)
+				)
+				(hide yes)
+			)
+		)
 		(pin "2"
 		)
@@
 			)
 		)
-		(property "Voltage" "10V"
+		(property "Voltage" "16V"
 			(at 147.828 78.994 0)
 			(effects
@@
 		)
 		(property "Function" "LED"
+			(at 143.51 76.2 0)
+			(effects
+				(font
+					(size 1.27 1.27)
+				)
+				(hide yes)
+			)
+		)
+		(property "LCSC Part #" "C1525"
+			(at 143.51 76.2 0)
+			(effects
+				(font
+					(size 1.27 1.27)
+				)
+				(hide yes)
+			)
+		)
+		(property "Manufacturer" "YAGEO"
 			(at 143.51 76.2 0)
 			(effects
@@
 			)
 		)
-		(property "Voltage" "10V"
+		(property "Voltage" "16V"
 			(at 187.198 78.994 0)
 			(effects
@@
 			(at 182.88 76.2 0)
 			(effects
+				(font
+					(size 1.27 1.27)
+				)
+				(hide yes)
+			)
+		)
+		(property "LCSC Part #" "C1525"
+			(at 182.88 76.2 0)
+			(effects
+				(font
+					(size 1.27 1.27)
+				)
+				(hide yes)
+			)
+		)
+		(property "Manufacturer" "YAGEO"
+			(at 182.88 76.2 0)
+			(effects

Commit message: prepare for the 1st test batch
Parts:
- renumbered C32 to C100, C33 to C101, C34 to C102, C31 to C99, LED2 to LED1, LED3 to LED2, LED4 to LED3, LED5 to LED4
Changed lines of the file:
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@@
 		(dnp no)
 		(fields_autoplaced yes)
-		(property "Reference" "#PWR065"
+		(property "Reference" "#PWR0191"
 			(at 182.88 72.39 0)
 			(effects
@@
 			(project ""
 				(path "/204e071a-14ed-47a0-be54-332ac2b951cf/18f90dfa-9bd7-48d0-80c5-47366522e296"
-					(reference "#PWR065")
+					(reference "#PWR0191")
 					(unit 1)
 				)
@@
 		(on_board yes)
 		(dnp no)
-		(property "Reference" "C31"
+		(property "Reference" "C99"
 			(at 105.156 73.66 0)
 			(effects
@@
 			(project ""
 				(path "/204e071a-14ed-47a0-be54-332ac2b951cf/18f90dfa-9bd7-48d0-80c5-47366522e296"
-					(reference "C31")
+					(reference "C99")
 					(unit 1)
 				)
@@
 		(dnp no)
 		(fields_autoplaced yes)
-		(property "Reference" "#PWR064"
+		(property "Reference" "#PWR0189"
 			(at 143.51 72.39 0)
 			(effects
@@
 			(project ""
 				(path "/204e071a-14ed-47a0-be54-332ac2b951cf/18f90dfa-9bd7-48d0-80c5-47366522e296"
-					(reference "#PWR064")
+					(reference "#PWR0189")
 					(unit 1)
 				)
@@
 		(dnp no)
 		(fields_autoplaced yes)
-		(property "Reference" "LED2"
+		(property "Reference" "LED1"
 			(at 85.09 63.5 0)
 			(effects
@@
 			(project ""
 				(path "/204e071a-14ed-47a0-be54-332ac2b951cf/18f90dfa-9bd7-48d0-80c5-47366522e296"
-					(reference "LED2")
+					(reference "LED1")
 					(unit 1)
 				)
@@
 		(dnp no)
 		(fields_autoplaced yes)
-		(property "Reference" "#PWR057"
+		(property "Reference" "#PWR0194"
 			(at 222.25 90.17 0)
 			(effects
@@
 			(project ""
 				(path "/204e071a-14ed-47a0-be54-332ac2b951cf/18f90dfa-9bd7-48d0-80c5-47366522e296"
-					(reference "#PWR057")
+					(reference "#PWR0194")
 					(unit 1)
 				)
@@
 		(dnp no)
 		(fields_autoplaced yes)
-		(property "Reference" "LED3"
+		(property "Reference" "LED2"
 			(at 125.73 63.5 0)
 			(effects
@@
 			(project "OBJ_PCB_onju_by_imike78_2025-05-11"
 				(path "/204e071a-14ed-47a0-be54-332ac2b951cf/18f90dfa-9bd7-48d0-80c5-47366522e296"
-					(reference "LED3")
+					(reference "LED2")
 					(unit 1)
 				)
@@
 		(dnp no)
 		(fields_autoplaced yes)
-		(property "Reference" "LED4"
+		(property "Reference" "LED3"
 			(at 165.1 63.5 0)
 			(effects
@@
 			(project "OBJ_PCB_onju_by_imike78_2025-05-11"
 				(path "/204e071a-14ed-47a0-be54-332ac2b951cf/18f90dfa-9bd7-48d0-80c5-47366522e296"
-					(reference "LED4")
+					(reference "LED3")
 					(unit 1)
 				)
@@
 		(on_board yes)
 		(dnp no)
-		(property "Reference" "C34"
+		(property "Reference" "C102"
 			(at 224.536 73.66 0)
 			(effects
@@
 			(project "OBJ_PCB_onju_by_imike78_2025-05-11"
 				(path "/204e071a-14ed-47a0-be54-332ac2b951cf/18f90dfa-9bd7-48d0-80c5-47366522e296"
-					(reference "C34")
+					(reference "C102")
 					(unit 1)
 				)
@@
 		(dnp no)
 		(fields_autoplaced yes)
-		(property "Reference" "#PWR061"
+		(property "Reference" "#PWR0188"
 			(at 102.87 90.17 0)
 			(effects
@@
 			(project ""
 				(path "/204e071a-14ed-47a0-be54-332ac2b951cf/18f90dfa-9bd7-48d0-80c5-47366522e296"
-					(reference "#PWR061")
+					(reference "#PWR0188")
 					(unit 1)
 				)
@@
 		(dnp no)
 		(fields_autoplaced yes)
-		(property "Reference" "LED5"
+		(property "Reference" "LED4"
 			(at 204.47 63.5 0)
 			(effects
@@
 			(project "OBJ_PCB_onju_by_imike78_2025-05-11"
 				(path "/204e071a-14ed-47a0-be54-332ac2b951cf/18f90dfa-9bd7-48d0-80c5-47366522e296"
-					(reference "LED5")
+					(reference "LED4")
 					(unit 1)
 				)
@@
 		(dnp no)
 		(fields_autoplaced yes)
-		(property "Reference" "#PWR060"
+		(property "Reference" "#PWR0190"
 			(at 143.51 90.17 0)
 			(effects
@@
 			(project ""
 				(path "/204e071a-14ed-47a0-be54-332ac2b951cf/18f90dfa-9bd7-48d0-80c5-47366522e296"
-					(reference "#PWR060")
+					(reference "#PWR0190")
 					(unit 1)
 				)
@@
 		(on_board yes)
 		(dnp no)
-		(property "Reference" "C32"
+		(property "Reference" "C100"
 			(at 145.796 73.66 0)
 			(effects
@@
 			(project "OBJ_PCB_onju_by_imike78_2025-05-11"
 				(path "/204e071a-14ed-47a0-be54-332ac2b951cf/18f90dfa-9bd7-48d0-80c5-47366522e296"
-					(reference "C32")
+					(reference "C100")
 					(unit 1)
 				)
@@
 		(dnp no)
 		(fields_autoplaced yes)
-		(property "Reference" "#PWR063"
+		(property "Reference" "#PWR0187"
 			(at 102.87 72.39 0)
 			(effects
@@
 			(project ""
 				(path "/204e071a-14ed-47a0-be54-332ac2b951cf/18f90dfa-9bd7-48d0-80c5-47366522e296"
-					(reference "#PWR063")
+					(reference "#PWR0187")
 					(unit 1)
 				)
@@
 		(dnp no)
 		(fields_autoplaced yes)
-		(property "Reference" "#PWR066"
+		(property "Reference" "#PWR0193"
 			(at 222.25 72.39 0)
 			(effects
@@
 			(project ""
 				(path "/204e071a-14ed-47a0-be54-332ac2b951cf/18f90dfa-9bd7-48d0-80c5-47366522e296"
-					(reference "#PWR066")
+					(reference "#PWR0193")
 					(unit 1)
 				)
@@
 		(on_board yes)
 		(dnp no)
-		(property "Reference" "C33"
+		(property "Reference" "C101"
 			(at 185.166 73.66 0)
 			(effects
@@
 			(project "OBJ_PCB_onju_by_imike78_2025-05-11"
 				(path "/204e071a-14ed-47a0-be54-332ac2b951cf/18f90dfa-9bd7-48d0-80c5-47366522e296"
-					(reference "C33")
+					(reference "C101")
 					(unit 1)
 				)
@@
 		(dnp no)
 		(fields_autoplaced yes)
-		(property "Reference" "#PWR058"
+		(property "Reference" "#PWR0192"
 			(at 182.88 90.17 0)
 			(effects
@@
 			(project ""
 				(path "/204e071a-14ed-47a0-be54-332ac2b951cf/18f90dfa-9bd7-48d0-80c5-47366522e296"
-					(reference "#PWR058")
+					(reference "#PWR0192")
 					(unit 1)
 				)

Commit message: prepare for the 1st test batch
Parts:
- renumbered C99 to C104, C100 to C105, C101 to C106, C102 to C107
Changed lines of the file:
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@@
 		(dnp no)
 		(fields_autoplaced yes)
-		(property "Reference" "#PWR0191"
+		(property "Reference" "#PWR0201"
 			(at 182.88 72.39 0)
 			(effects
@@
 			(project ""
 				(path "/204e071a-14ed-47a0-be54-332ac2b951cf/18f90dfa-9bd7-48d0-80c5-47366522e296"
-					(reference "#PWR0191")
+					(reference "#PWR0201")
 					(unit 1)
 				)
@@
 		(on_board yes)
 		(dnp no)
-		(property "Reference" "C99"
+		(property "Reference" "C104"
 			(at 105.156 73.66 0)
 			(effects
@@
 			(project ""
 				(path "/204e071a-14ed-47a0-be54-332ac2b951cf/18f90dfa-9bd7-48d0-80c5-47366522e296"
-					(reference "C99")
+					(reference "C104")
 					(unit 1)
 				)
@@
 		(dnp no)
 		(fields_autoplaced yes)
-		(property "Reference" "#PWR0189"
+		(property "Reference" "#PWR0199"
 			(at 143.51 72.39 0)
 			(effects
@@
 			(project ""
 				(path "/204e071a-14ed-47a0-be54-332ac2b951cf/18f90dfa-9bd7-48d0-80c5-47366522e296"
-					(reference "#PWR0189")
+					(reference "#PWR0199")
 					(unit 1)
 				)
@@
 		(dnp no)
 		(fields_autoplaced yes)
-		(property "Reference" "#PWR0194"
+		(property "Reference" "#PWR0204"
 			(at 222.25 90.17 0)
 			(effects
@@
 			(project ""
 				(path "/204e071a-14ed-47a0-be54-332ac2b951cf/18f90dfa-9bd7-48d0-80c5-47366522e296"
-					(reference "#PWR0194")
+					(reference "#PWR0204")
 					(unit 1)
 				)
@@
 		(on_board yes)
 		(dnp no)
-		(property "Reference" "C102"
+		(property "Reference" "C107"
 			(at 224.536 73.66 0)
 			(effects
@@
 			(project "OBJ_PCB_onju_by_imike78_2025-05-11"
 				(path "/204e071a-14ed-47a0-be54-332ac2b951cf/18f90dfa-9bd7-48d0-80c5-47366522e296"
-					(reference "C102")
+					(reference "C107")
 					(unit 1)
 				)
@@
 		(dnp no)
 		(fields_autoplaced yes)
-		(property "Reference" "#PWR0188"
+		(property "Reference" "#PWR0198"
 			(at 102.87 90.17 0)
 			(effects
@@
 			(project ""
 				(path "/204e071a-14ed-47a0-be54-332ac2b951cf/18f90dfa-9bd7-48d0-80c5-47366522e296"
-					(reference "#PWR0188")
+					(reference "#PWR0198")
 					(unit 1)
 				)
@@
 		(dnp no)
 		(fields_autoplaced yes)
-		(property "Reference" "#PWR0190"
+		(property "Reference" "#PWR0200"
 			(at 143.51 90.17 0)
 			(effects
@@
 			(project ""
 				(path "/204e071a-14ed-47a0-be54-332ac2b951cf/18f90dfa-9bd7-48d0-80c5-47366522e296"
-					(reference "#PWR0190")
+					(reference "#PWR0200")
 					(unit 1)
 				)
@@
 		(on_board yes)
 		(dnp no)
-		(property "Reference" "C100"
+		(property "Reference" "C105"
 			(at 145.796 73.66 0)
 			(effects
@@
 			(project "OBJ_PCB_onju_by_imike78_2025-05-11"
 				(path "/204e071a-14ed-47a0-be54-332ac2b951cf/18f90dfa-9bd7-48d0-80c5-47366522e296"
-					(reference "C100")
+					(reference "C105")
 					(unit 1)
 				)
@@
 		(dnp no)
 		(fields_autoplaced yes)
-		(property "Reference" "#PWR0187"
+		(property "Reference" "#PWR0197"
 			(at 102.87 72.39 0)
 			(effects
@@
 			(project ""
 				(path "/204e071a-14ed-47a0-be54-332ac2b951cf/18f90dfa-9bd7-48d0-80c5-47366522e296"
-					(reference "#PWR0187")
+					(reference "#PWR0197")
 					(unit 1)
 				)
@@
 		(dnp no)
 		(fields_autoplaced yes)
-		(property "Reference" "#PWR0193"
+		(property "Reference" "#PWR0203"
 			(at 222.25 72.39 0)
 			(effects
@@
 			(project ""
 				(path "/204e071a-14ed-47a0-be54-332ac2b951cf/18f90dfa-9bd7-48d0-80c5-47366522e296"
-					(reference "#PWR0193")
+					(reference "#PWR0203")
 					(unit 1)
 				)
@@
 		(on_board yes)
 		(dnp no)
-		(property "Reference" "C101"
+		(property "Reference" "C106"
 			(at 185.166 73.66 0)
 			(effects
@@
 			(project "OBJ_PCB_onju_by_imike78_2025-05-11"
 				(path "/204e071a-14ed-47a0-be54-332ac2b951cf/18f90dfa-9bd7-48d0-80c5-47366522e296"
-					(reference "C101")
+					(reference "C106")
 					(unit 1)
 				)
@@
 		(dnp no)
 		(fields_autoplaced yes)
-		(property "Reference" "#PWR0192"
+		(property "Reference" "#PWR0202"
 			(at 182.88 90.17 0)
 			(effects
@@
 			(project ""
 				(path "/204e071a-14ed-47a0-be54-332ac2b951cf/18f90dfa-9bd7-48d0-80c5-47366522e296"
-					(reference "#PWR0192")
+					(reference "#PWR0202")
 					(unit 1)
 				)

Commit message: ready for the 1st test batch
Parts:
- C104, C105, C106, C107: Manufacturer YAGEO -> Samsung Electro-Mechanics; Manufacturer Part (none) -> CL05B104KO5NNNC
Changed lines of the file:
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@@
 			)
 		)
-		(property "Manufacturer" "YAGEO"
+		(property "Manufacturer" "Samsung Electro-Mechanics"
 			(at 102.87 76.2 0)
 			(effects
@@
 		)
 		(property "CL" ""
+			(at 102.87 76.2 0)
+			(effects
+				(font
+					(size 1.27 1.27)
+				)
+				(hide yes)
+			)
+		)
+		(property "Manufacturer Part" "CL05B104KO5NNNC"
 			(at 102.87 76.2 0)
 			(effects
@@
 			)
 		)
-		(property "Manufacturer" "YAGEO"
+		(property "Manufacturer" "Samsung Electro-Mechanics"
 			(at 222.25 76.2 0)
 			(effects
@@
 		)
 		(property "CL" ""
+			(at 222.25 76.2 0)
+			(effects
+				(font
+					(size 1.27 1.27)
+				)
+				(hide yes)
+			)
+		)
+		(property "Manufacturer Part" "CL05B104KO5NNNC"
 			(at 222.25 76.2 0)
 			(effects
@@
 			)
 		)
-		(property "Manufacturer" "YAGEO"
+		(property "Manufacturer" "Samsung Electro-Mechanics"
 			(at 143.51 76.2 0)
 			(effects
@@
 		)
 		(property "CL" ""
+			(at 143.51 76.2 0)
+			(effects
+				(font
+					(size 1.27 1.27)
+				)
+				(hide yes)
+			)
+		)
+		(property "Manufacturer Part" "CL05B104KO5NNNC"
 			(at 143.51 76.2 0)
 			(effects
@@
 			)
 		)
-		(property "Manufacturer" "YAGEO"
+		(property "Manufacturer" "Samsung Electro-Mechanics"
 			(at 182.88 76.2 0)
 			(effects
@@
 			(at 182.88 76.2 0)
 			(effects
+				(font
+					(size 1.27 1.27)
+				)
+				(hide yes)
+			)
+		)
+		(property "Manufacturer Part" "CL05B104KO5NNNC"
+			(at 182.88 76.2 0)
+			(effects
