File: leds.kicad_sch (KiCad schematic)
At the start: 8 parts

Commit message: v2 hardware revision
MPR121 touch controller added to replace esp32-s3 integrated touch pins
Parts:
- LED1, LED2, LED3, LED4: Availability Not in stock -> (none); Check_prices https://www.snapeda.com/parts/SK6812-E/DONGGUANG+OPSCO+OPTO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 -> (none); PARTREV 2 -> (none)
