File: home-mini-DiP-v1.kicad_pcb (KiCad board)
At the start: 4 copper layers, 72.4 x 70 mm, 241 parts, among them J1 FH34SRJ-16S-0.5SH_50_, J2 1775443-2, J3 XMOS JTAG, J4 XTAG DEV, J5 Conn_01x05, Q1 LBSS138WT1G, Q2 LBSS138WT1G, Q3 BC847B, SW2 BOOT, U1 AP22802AW5-7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

Commit message: production update + esphome fw update + latest render pics
Parts:
- moved X1 3.10 mm to (136.9, 79.2)
